File: BatteryBank.kicad_sch (KiCad schematic)
At the start: 138 parts, among them J1 12402082E512A, J2 12402082E512A, Q1 40V N-FET TBD, buck high, Q2 40V N-FET TBD, buck low, Q3 40V N-FET TBD, boost low, Q4 40V N-FET TBD, boost high, Q5 30V N-FET TBD, discharge, Q6 30V N-FET TBD, charge, U1 TPS25751D, U2 BQ25756, U3 24C-series EEPROM (TBD), U4 BQ7791501, U5 TPS70933DBV, U6 TPS62933, U7 STM32WB1MMC, U8 TPS25810

Commit message: Draft 5: parts selected, real pin numbers, standard footprints
- FETs: AGM404AP1 (JLC C41349455) in all six positions
- Inductors: Sunlord MWSA1004S-3R3MT and MWSA0603S-3R3MT
- EEPROM: BL24C512A, 8-pin symbol
- Port 1 ESD protection added (PESD24VS2UT, PESD5V0S2UT)
- LCSC part numbers stored on parts where known
- Standard footprints assigned to 119 of 141 parts

Co-Authored-By: Claude Opus 5.5 <noreply@anthropic.com>
Claude-Session: https://claude.ai/code/session_017ypupkahdxpHbW4uwEu58x
Parts:
- removed U3: 24C-series EEPROM (TBD), symbol Monolith:EEPROM_I2C
- added C59: 100n, Capacitor_SMD:C_0402_1005Metric, symbol Monolith:C
- added D3: PESD24VS2UT, Package_TO_SOT_SMD:SOT-23, symbol Monolith:ESD_DUAL
- added D4: PESD5V0S2UT, Package_TO_SOT_SMD:SOT-23, symbol Monolith:ESD_DUAL
- added U3: BL24C512A-SFRC, Package_SO:TSSOP-8_4.4x3mm_P0.65mm, symbol Monolith:EEPROM_24C512
- C1, C2, C21, C22, C42, C43, C44, C47, C50, C55, C57, C58: footprint (none) -> Capacitor_SMD:C_0402_1005Metric
- C11, C12, C13, C14, C6, C7, C8, C9: footprint (none) -> Capacitor_SMD:C_1210_3225Metric
- C16, C17, C18, C3, C30, C31, C32, C33, C34, C35, C4, C40, C41, C5, C51, C56: footprint (none) -> Capacitor_SMD:C_0603_1608Metric
- C19, C20, C48, C49: footprint (none) -> Capacitor_SMD:C_0805_2012Metric
- C45, C46: footprint (none) -> Capacitor_SMD:C_1206_3216Metric
- D10, D11, D12, D13: footprint (none) -> LED_SMD:LED_0603_1608Metric
- L1: value 4.7uH 12A TBD -> 3.3uH MWSA1004S-3R3MT
- L2: value 3.3uH 5A -> 3.3uH MWSA0603S-3R3MT; LCSC (none) -> C408446
- Q1: value 40V N-FET TBD, buck high -> AGM404AP1, buck high; LCSC (none) -> C41349455; Status part to be selected -> 40V 4.4mOhm at 10V, PDFN 3.3x3.3; pinout to confirm in data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
- Q2: value 40V N-FET TBD, buck low -> AGM404AP1, buck low; LCSC (none) -> C41349455; Status part to be selected -> 40V 4.4mOhm at 10V, PDFN 3.3x3.3; pinout to confirm in data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
- Q3: value 40V N-FET TBD, boost low -> AGM404AP1, boost low; LCSC (none) -> C41349455; Status part to be selected -> 40V 4.4mOhm at 10V, PDFN 3.3x3.3; pinout to confirm in data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
- Q4: value 40V N-FET TBD, boost high -> AGM404AP1, boost high; LCSC (none) -> C41349455; Status part to be selected -> 40V 4.4mOhm at 10V, PDFN 3.3x3.3; pinout to confirm in data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
- Q5: value 30V N-FET TBD, discharge -> AGM404AP1, discharge; LCSC (none) -> C41349455; Status part to be selected -> 40V 4.4mOhm at 10V, PDFN 3.3x3.3; pinout to confirm in data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
- Q6: value 30V N-FET TBD, charge -> AGM404AP1, charge; LCSC (none) -> C41349455; Status part to be selected -> 40V 4.4mOhm at 10V, PDFN 3.3x3.3; pinout to confirm in data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
- R1, R2, R36: footprint (none) -> Resistor_SMD:R_2512_6332Metric
- R10, R11, R12, R13, R14, R15, R16, R17, R18, R19, R20, R21, R22, R23, R24, R25, R26, R27, R3, R30, R31, R32, R33, R34, R35, R37, R38, R39, R4, R40, R41, R42, R43, R44, R45, R46, R47, R48, R49, R5, R50, R51, R52, R53, R54, R55, R56, R6, R7, R8, R9: footprint (none) -> Resistor_SMD:R_0402_1005Metric
- U2: LCSC (none) -> C19272232
- U4: footprint (none) -> Package_SO:TSSOP-24_4.4x7.8mm_P0.65mm
- U5: footprint (none) -> Package_TO_SOT_SMD:SOT-23-5; LCSC (none) -> C89347
- U6: footprint (none) -> Package_TO_SOT_SMD:SOT-583-8
- U8: LCSC (none) -> C473913
- W1, W2, W3, W4, W5: footprint (none) -> TestPoint:TestPoint_Pad_4.0x4.0mm
- W10, W11, W12, W6, W7, W8, W9: footprint (none) -> TestPoint:TestPoint_Pad_D1.5mm
Connections:
- net AC_SNS_N: now also Q1.5 (D), Q1.6 (D), Q1.7 (D), Q1.8 (D); no longer Q1.D
- net BAT_SNS_P: now also Q4.5 (D), Q4.6 (D), Q4.7 (D), Q4.8 (D); no longer Q4.D
- net CHG_SCL: now also U3.6 (SCL)
- net CHG_SDA: now also U3.5 (SDA)
- net GND: now also Q2.1 (S), Q2.2 (S), Q2.3 (S), Q3.1 (S), Q3.2 (S), Q3.3 (S), Q6.1 (S), Q6.2 (S), Q6.3 (S), C59.2, D3.3 (A), D4.3 (A), U3.1 (A0), U3.2 (A1), U3.3 (A2), U3.4 (VSS), U3.7 (WP); no longer Q2.S, Q3.S, Q6.S
- net HG1: now also Q1.4 (G); no longer Q1.G
- net HG2: now also Q4.4 (G); no longer Q4.G
- net LG1: now also Q2.4 (G); no longer Q2.G
- net LG2: now also Q3.4 (G); no longer Q3.G
- net P1_CC1: now also D3.1 (K1)
- net P1_CC2: now also D3.2 (K2)
- net P1_DN: now also D4.2 (K2)
- net P1_DP: now also D4.1 (K1)
- net PD_3V3: now also C59.1, U3.8 (VCC)
- net PROT_CHG_G: now also Q6.4 (G); no longer Q6.G
- net PROT_DSG_G: now also Q5.4 (G); no longer Q5.G
- net PROT_MID: now also Q5.5 (D), Q5.6 (D), Q5.7 (D), Q5.8 (D), Q6.5 (D), Q6.6 (D), Q6.7 (D), Q6.8 (D); no longer Q5.D, Q6.D
- net PROT_SNS: now also Q5.1 (S), Q5.2 (S), Q5.3 (S); no longer Q5.S
- net SW1: now also Q1.1 (S), Q1.2 (S), Q1.3 (S), Q2.5 (D), Q2.6 (D), Q2.7 (D), Q2.8 (D); no longer Q1.S, Q2.D
- net SW2: now also Q3.5 (D), Q3.6 (D), Q3.7 (D), Q3.8 (D), Q4.1 (S), Q4.2 (S), Q4.3 (S); no longer Q3.D, Q4.S
Other:
- note added: "Connections are made by net labels at each pin. Resistors marked TBD still need values. Standard footprints are assigned; custom packages are still blank."
- note added: "Monolith top board: all blocks. DRAFT 5, generated from the TI pin tables."
- note removed: "Connections are made by net labels at each pin. Parts marked TBD are not final. Port 1 ESD protection is not drawn yet."
- note removed: "Monolith top board: all blocks. DRAFT 3, generated from the TI pin tables."

Commit message: Draft 6: datasheet corrections to charger and PD controller wiring
- Fix ACUV/ACOV divider order (VAC > ACUV > ACOV > GND) and set values
  for a 4.4 V to 24 V input window (1M / 267k / 66.5k)
- Charge voltage divider now 249k / 25.5k per TI's equation (16.5 V)
- TPS25751 boot strap: ADCIN1 to LDO_3V3, ADCIN2 to GND (SafeMode),
  strap resistors removed
- Note I2C addresses on the sheet

Co-Authored-By: Claude Opus 5.5 <noreply@anthropic.com>
Claude-Session: https://claude.ai/code/session_017ypupkahdxpHbW4uwEu58x
Parts:
- removed R24, R25, R26, R27: TBD, Resistor_SMD:R_0402_1005Metric, symbol Monolith:R
- R11: value TBD -> 1M 1%; Status value to be set -> value to confirm
- R12: value TBD -> 267k 1%; Status value to be set -> value to confirm
- R13: value TBD -> 66.5k 1%; Status value to be set -> value to confirm
- R4: value 243k 0.1% -> 249k 0.1%
- R5: value 24.9k 0.1% -> 25.5k 0.1%
- U1: Status pinout from TI datasheet -> pinout and boot strap from TI datasheet
Connections:
- net ADCIN1 is gone; now on net PD_3V3: U1.2 (ADCIN1)
- net ADCIN2 is gone; now on net GND: U1.3 (ADCIN2)
- net CHG_ACOV: now also R12.2, R13.1; no longer R11.2, R12.1
- net CHG_ACUV: now also R11.2, R12.1; no longer R12.2, R13.1
Other:
- note added: "I2C addresses on the charger bus: BQ25756 0x6B, EEPROM 0x50. Charge voltage 16.5V, charge current 3A, input window 4.4V to 24V, 400kHz."
- note added: "Monolith top board: all blocks. DRAFT 6, generated from the TI pin tables."
- note removed: "Monolith top board: all blocks. DRAFT 5, generated from the TI pin tables."
