File: DevBoard/usb_port.kicad_sch (KiCad schematic)
At the start: 101 parts, among them J501 TYPE-C 16PCB0.8 IP68, J502 I2CC logic analyzer, Q501 IAUC45N04S6L063H, Q502 IAUC45N04S6L063H, U501 TPS25751DREFR, U502 M24512-DFMC6TG, U503 BQ25756RRVR, U504 TPS62933DRLR

Commit message: Dev board rev A5: BAT fed before F101, review 2 hardware fixes, JLC passives
- Gauge BAT feed follows TI fig. 9-12: D101 from the cell top (CELL_P_RAW)
  before F101, so the gauge stays powered if the fuse opens or is unfitted.
- C421/C521 100 uF 35 V polymer (same 6.3 mm footprint): about 99 uF worst
  case vs the BQ25756 80 uF minimum after derating.
- Bootstrap diodes LRB520S-40T1G, Q103 BSS138, DNP C109 4.7 nF (fit D103
  with it), PPHV 0.1 uF and VBUS 10 nF per port, R306 330R, C201 DNP flag.
- Test points: GND loops by each port's SW probes and in the pack probe
  field, CELL_P_RAW, CE_N, LDO_3V3, LDO_IN, 5V_AMP.
- JLC part numbers on every resistor and capacitor.
- Placement for the new parts; placer hides test-point labels with no
  free spot. DRC clean, schematic parity clean.

Co-Authored-By: Claude Opus 5.5 <noreply@anthropic.com>
Parts:
- added C549: 0.1u 50V, Capacitor_SMD:C_0603_1608Metric, symbol Device:C
- added C550: 10n 50V, Capacitor_SMD:C_0603_1608Metric, symbol Device:C
- added TP512: GND, TestPoint:TestPoint_Keystone_5000-5004_Miniature, symbol Connector:TestPoint
- added TP513: CE_N, TestPoint:TestPoint_Pad_D1.5mm, symbol Connector:TestPoint
- added TP514: LDO_3V3, TestPoint:TestPoint_Pad_D1.5mm, symbol Connector:TestPoint
- C507: value 10u 10V -> 10u 25V; LCSC (none) -> C15850; MPN (none) -> CL21A106KAYNNNE
- C510, C511: value 4.7u 16V -> 4.7u 25V; LCSC (none) -> C1779; MPN (none) -> CL21A475KAQNNNE
- C512, C513, C540: value 0.1u 25V -> 0.1u 50V; LCSC (none) -> C14663; MPN (none) -> CC0603KRX7R9BB104
- C514, C517: LCSC (none) -> C1623; MPN (none) -> CL10B474KA8NNNC
- C515, C516, C518, C519, C530, C538, C546: LCSC (none) -> C14663; MPN (none) -> CC0603KRX7R9BB104
- C521: value 68u 35V -> 100u 35V; footprint Capacitor_SMD:CP_Elec_6.3x5.8 -> Capacitor_SMD:CP_Elec_6.3x7.7; LCSC C49435121 -> C5246554; MPN ChuangHui SV680M350E5R8R4Z00ZZ (polymer) -> Honor Elec HV1V107M0607PZ (polymer); Notes USB-side bulk: solid polymer, no DC-bias loss (68 uF at 20 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 -> USB-side bulk, polymer (no DC-bias loss). 100 uF (was 68 uF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
- C539: value 33n -> 33n 50V; LCSC (none) -> C21117; MPN (none) -> CL10B333KB8NNNC
- C541, C542: value 22u 35V -> 22u 25V; LCSC (none) -> C12891; MPN (none) -> CL31A226KAHNNNE
- C544, C545: LCSC (none) -> C13585; MPN (none) -> CL31A106KBHNNNE
- D504: value LRB521S-40 -> LRB520S-40T1G; LCSC C135802 -> C132124; MPN LRB521S-40T1G (LRC) -> LRB520S-40T1G; Notes Bootstrap diode DRV_SUP -> BTST1 (Q401 high side). TI BQ257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 -> Bootstrap diode DRV_SUP -> BTST (TI BQ25756 checklist: requ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
- D505: value LRB521S-40 -> LRB520S-40T1G; LCSC C135802 -> C132124; MPN LRB521S-40T1G (LRC) -> LRB520S-40T1G; Notes Bootstrap diode DRV_SUP -> BTST2 (Q402 high side). TI BQ257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 -> Bootstrap diode DRV_SUP -> BTST (TI BQ25756 checklist: requ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
- R501: LCSC (none) -> C17477; MPN (none) -> 0805W8F0000T5E
- R502, R503: LCSC (none) -> C22978; MPN (none) -> 0603WAF3301T5E
- R504, R521, R522, R523: LCSC (none) -> C25804; MPN (none) -> 0603WAF1002T5E
- R520, R525, R526, R528, R529: LCSC (none) -> C22859; MPN (none) -> 0603WAF100JT5E
- R532: LCSC (none) -> C25803; MPN (none) -> 0603WAF1003T5E
Connections:
- net CE_N: now also TP513.1
- net GND: now also C549.2, C550.2, TP512.1
- net LDO_3V3: now also TP514.1
- net PPHV: now also C549.1
- net VBUS: now also C550.1

Commit message: Dev board: SMD test loops (RH-S2761-46R) instead of Keystone through-hole
All 45 loop test points become ronghe RH-S2761-46R (LCSC C55121754), the
JLC-stocked equivalent of the Harwin S2761-46R: 1.6 x 0.8 x 1.15 mm SMT
loop on an 0603 land pattern, 3.5 A. New footprint
MonolithDev:TestPoint_Harwin_S2761_0603 (make_footprints.py section 11),
both pads pin 1 and jumpered. JLC places them; no through-hole assembly.

Co-Authored-By: Claude Opus 5.5 <noreply@anthropic.com>
Parts:
- TP501, TP502, TP503, TP504, TP505, TP506, TP507, TP508, TP509, TP510, TP511, TP512: footprint TestPoint:TestPoint_Keystone_5000-5004_Miniature -> MonolithDev:TestPoint_Harwin_S2761_0603; LCSC (none) -> C55121754; MPN (none) -> RH-S2761-46R (ronghe; Harwin S2761-46R equivalent)

Commit message: Dev board: open-item pass, J104 diode, antenna keep-out, bring-up checklist
- D104 SS34 in series with the J104 bench input (reversed lead, back-feed).
- ANT_KEEPOUT rule area (no tracks/vias/pours, all copper layers) around
  the STM32WB1MMC antenna end, created by place_parts.py.
- D401 drawn unidirectional; header part numbers (PZ254V-11 family);
  shunt, J301 keying, B-constant, insulated-NTC, sheet-text and R201 notes.
- docs/devboard/bringup-config-checklist.md: every configuration item from
  both reviews in bring-up order, with review 2's precharge correction;
  review 1's 0 mV precharge line marked superseded.

Co-Authored-By: Claude Opus 5.5 <noreply@anthropic.com>
Parts:
- D501: symbol Device:D_TVS -> Device:D_Zener; Notes (none) -> SMAJ22A is unidirectional: drawn as a zener-style TVS, cath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
- J502: LCSC (none) -> C2937625; MPN (none) -> PZ254V-11-03P
- TH501: Notes beside FETs -> beside FETs. Murata NCP18XH103F03RB: B25/50 = 3380 K, B25/8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
Other:
- note added: "BQ25756 CONTROLLER (600 kHz, ICHG 5.5 A max, ILIM 5.6 A, VAC 4.1-22.5 V window)"
- note added: "PP5V SUPPLY TPS62933 (1.2 MHz, 5.08 V) - 5 V source + VCONN"
- note removed: "BQ25756 CONTROLLER (600 kHz, ICHG 5.5 A max, ILIM 5.5 A, VAC 4.1-22.5 V window)"
- note removed: "PP5V SUPPLY TPS62933 (1.2 MHz, 5.00 V) - 5 V source + VCONN"
Changed lines of the file:
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@@
 		(comment 3 "Not reviewed, laid out, built or tested")
 	)
-	(text "PP5V SUPPLY  TPS62933 (1.2 MHz, 5.00 V)  - 5 V source + VCONN"
+	(text "PP5V SUPPLY  TPS62933 (1.2 MHz, 5.08 V)  - 5 V source + VCONN"
 		(exclude_from_sim no)
 		(at 40.64 182.88 0)
@@
 		)
 	)
-	(text "BQ25756 CONTROLLER  (600 kHz, ICHG 5.5 A max, ILIM 5.5 A, VAC 4.1-22.5 V window)"
+	(text "BQ25756 CONTROLLER  (600 kHz, ICHG 5.5 A max, ILIM 5.6 A, VAC 4.1-22.5 V window)"
 		(exclude_from_sim no)
 		(at 304.8 167.64 0)
@@
 			)
 		)
+		(property "LCSC" "C2937625"
+			(at 284.48 152.4 0)
+			(hide yes)
+			(show_name no)
+			(do_not_autoplace no)
+			(effects
+				(font
+					(size 1.27 1.27)
+				)
+			)
+		)
+		(property "MPN" "PZ254V-11-03P"
+			(at 284.48 152.4 0)
+			(hide yes)
+			(show_name no)
+			(do_not_autoplace no)
+			(effects
+				(font
+					(size 1.27 1.27)
+				)
+			)
+		)
 		(pin "1"
 		)
@@
 	)
 	(symbol
-		(lib_id "Device:D_TVS")
+		(lib_id "Device:D_Zener")
 		(at 73.66 88.9 270)
 		(unit 1)
@@
 			)
 		)
+		(property "Notes" "SMAJ22A is unidirectional: drawn as a zener-style TVS, cathode (pin 1) on VBUS"
+			(at 73.66 88.9 0)
+			(hide yes)
+			(show_name no)
+			(do_not_autoplace no)
+			(effects
+				(font
+					(size 1.27 1.27)
+				)
+			)
+		)
 		(pin "1"
 		)
@@
 			)
 		)
-		(property "Notes" "beside FETs"
+		(property "Notes" "beside FETs. Murata NCP18XH103F03RB: B25/50 = 3380 K, B25/85 = 3435 K (the \"B3435\" in the value); use Murata's R-T table in firmware and in the TS divider math"
 			(at 86.36 -3.81 0)
 			(hide yes)

Commit message: Dev board: accept holder contact resistance; record C421 ESR/ripple check
- Review 1 #4 marked accepted for rev 1 (BH-21700-B1BJ001, 100 mOhm max per
  holder); measure each holder at bring-up, holder mode about 2 A, heavy
  tests on the welded pack via J101.
- C421/C521 (HV1V107M0607PZ): datasheet ESR 48 mOhm, 1.5 A rms. Worst-case
  bank ripple about 5 A rms in reverse mode; the MLCCs take about 80 %, so
  the polymer sees about 1 A rms.

Co-Authored-By: Claude Opus 5.5 <noreply@anthropic.com>
Parts:
- C521: Notes USB-side bulk, polymer (no DC-bias loss). 100 uF (was 68 uF, review 2 B-5): MLCCs keep only ~6 uF each at 20 V, so 68 uF left 72-75 uF worst case vs the BQ25756 80 uF minimum after derating; now ~99 uF. Same 6.3 mm footprint, 7.7 mm tall. Check ESR/ripple in the maker datasheet (not listed at JLC) -> USB-side bulk, polymer (no DC-bias loss). 100 uF (was 68 uF, review 2 B-5): ~99 uF worst case vs the BQ25756 80 uF minimum after derating. Datasheet: ESR 48 mOhm, ripple 1.5 A rms. Worst-case bank ripple ~5 A rms (reverse mode, 10 V pack to 20 V 5 A); the four 22 uF MLCCs (~11 mOhm at 600 kHz) take ~80 %, so this cap sees ~1 A rms (~50 mW). Same 6.3 mm footprint, 7.7 mm tall
Changed lines of the file:
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@@
 			)
 		)
-		(property "Notes" "USB-side bulk, polymer (no DC-bias loss). 100 uF (was 68 uF, review 2 B-5): MLCCs keep only ~6 uF each at 20 V, so 68 uF left 72-75 uF worst case vs the BQ25756 80 uF minimum after derating; now ~99 uF. Same 6.3 mm footprint, 7.7 mm tall. Check ESR/ripple in the maker datasheet (not listed at JLC)"
+		(property "Notes" "USB-side bulk, polymer (no DC-bias loss). 100 uF (was 68 uF, review 2 B-5): ~99 uF worst case vs the BQ25756 80 uF minimum after derating. Datasheet: ESR 48 mOhm, ripple 1.5 A rms. Worst-case bank ripple ~5 A rms (reverse mode, 10 V pack to 20 V 5 A); the four 22 uF MLCCs (~11 mOhm at 600 kHz) take ~80 %, so this cap sees ~1 A rms (~50 mW). Same 6.3 mm footprint, 7.7 mm tall"
 			(at 327.66 121.92 0)
 			(hide yes)

Commit message: Dev board: start routing - planes, port power stages, gate drive, USB-C path, 5 V bucks
- Kelvin net class (0.2 mm / 0.15 mm) for the sense nets.
- tools/route_power.py (re-runnable, uuid sidecar): per port SW1/SW2 pours,
  input/output bank pours on F.Cu+B.Cu with GND islands stitched to In1,
  VBAT_SYS, gate drive on In2/B.Cu with F.Cu bootstrap loops, BQ25756 EP vias,
  VBUS and PPHV power path with RAC Kelvin taps, TPS62933 5 V buck and the
  PP5V feed to the TPS25751. In1 solid GND, In2 GND fill, M3 hole keep-outs.
- Placement: RBAT turned 180, SRP/SRN resistors beside it, gate-drive support
  parts regrouped ("fix" entries), C407/C507 0805 -> 0603 (CL10A106MA8NRNC,
  C96446) moved above U401 off the VBUS power pad.
- TPS25751 footprint: exposed-pad thermal vias solid to the planes.
- DRC 0 violations. README item 32.

Co-Authored-By: Claude Opus 5.5 <noreply@anthropic.com>
Parts:
- C507: footprint Capacitor_SMD:C_0805_2012Metric -> Capacitor_SMD:C_0603_1608Metric; LCSC C15850 -> C96446; MPN CL21A106KAYNNNE -> CL10A106MA8NRNC; Notes at PP5V pin -> at PP5V pin (0603: sits between U401 and its strap resistor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
Changed lines of the file:
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@@
 			)
 		)
-		(property "Footprint" "Capacitor_SMD:C_0805_2012Metric"
+		(property "Footprint" "Capacitor_SMD:C_0603_1608Metric"
 			(at 237.185 67.31 0)
 			(hide yes)
@@
 			)
 		)
-		(property "Notes" "at PP5V pin"
+		(property "Notes" "at PP5V pin (0603: sits between U401 and its strap resistors, clear of the VBUS power pad)"
 			(at 7.62 0 0)
 			(hide yes)
@@
 			)
 		)
-		(property "LCSC" "C15850"
+		(property "LCSC" "C96446"
 			(at 236.22 71.12 0)
 			(hide yes)
@@
 			)
 		)
-		(property "MPN" "CL21A106KAYNNNE"
+		(property "MPN" "CL10A106MA8NRNC"
 			(at 236.22 71.12 0)
 			(hide yes)

Commit message: Dev board: second-level pack protection, D103 fitted, U202 JLC, strap cleanup
- Gauge sheet: BQ294700 (4.35 V/cell OVP) and the BQ40Z50 FUSE pin share
  ignition FET Q104 (TI BQ40Z50-R2 fig. 9-11) to blow F102, a TLC WSFB1514
  4-cell 15 A self-control fuse at the cell top. F101 removed: F102 is the
  pack fuse. R127 DNP bench bypass. New symbols/footprint/3D model.
- D103 (Q102 gate-source 15 V clamp) fitted on dev board and production.
- U202 INA190A1 now JLC-assembled (C1852068); U201 stays hand-soldered.
- TPS25751 ADCIN divider footprints R405-R408 removed (SafeMode 0x20/0x21
  needs only the R1-R4 ties); place_parts rows and notes updated.
- Layout not yet updated for these changes.

Co-Authored-By: Claude Opus 5.5 <noreply@anthropic.com>
Parts:
- removed R505, R506, R507, R508: DNP, Resistor_SMD:R_0603_1608Metric, symbol Device:R
- renumbered C501 to C401, C502 to C402, C503 to C403, C504 to C404, C505 to C405, C506 to C406, C507 to C407, C508 to C408, C509 to C409, C510 to C410, C511 to C411, C512 to C412, C513 to C413, C514 to C414, C515 to C415, C516 to C416, C517 to C417, C518 to C418, C519 to C419, C520 to C420, C521 to C421, C523 to C423, C524 to C424, C527 to C427, C530 to C430, C531 to C431, C532 to C432, C534 to C434, C535 to C435, C538 to C438, C539 to C439, C540 to C440, C541 to C441, C542 to C442, C543 to C443, C544 to C444, C545 to C445, C546 to C446, C547 to C447, C549 to C449, C550 to C450, D501 to D401, D502 to D402, D503 to D403, D504 to D404, D505 to D405, J501 to J401, J502 to J402, L501 to L401, L502 to L402, Q501 to Q401, Q502 to Q402, R501 to R401, R502 to R402, R503 to R403, R504 to R404, R509 to R409, R510 to R410, R511 to R411, R512 to R412, R513 to R413, R514 to R414, R515 to R415, R516 to R416, R517 to R417, R518 to R418, R519 to R419, R520 to R420, R521 to R421, R522 to R422, R523 to R423, R524 to R424, R525 to R425, R526 to R426, R527 to R427, R528 to R428, R529 to R429, R530 to R430, R531 to R431, R532 to R432, R533 to R433, R534 to R434, R535 to R435, TH501 to TH401, TP501 to TP401, TP502 to TP402, TP503 to TP403, TP504 to TP404, TP505 to TP405, TP506 to TP406, TP507 to TP407, TP508 to TP408, TP509 to TP409, TP510 to TP410, TP511 to TP411, TP512 to TP412, TP513 to TP413, TP514 to TP414, U501 to U401, U502 to U402, U503 to U403, U504 to U404
Other:
- note added: "NOTES (this sheet is used twice: USB Port 1 = 4xx, USB Port 2 = 5xx) 1. Address straps are on the root sheet: port 1 ADCIN1 = LDO_3V3, ADCIN2 = GND (0x20); port 2 ADCIN1 = ADCIN2 = GND (0x21). Both are SafeMode (TPS25751 table 8-6). 2. Unused TPS25751 GPIOs tied to GND per datasheet (KiCad ERC flags this; expected). 3. At the connector pins: D402 CC ESD (24 V), D403 D+/D- ESD (5 V: GPIO4/5 are ra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"
- note removed: "NOTES (this sheet is used twice: USB Port 1 = 4xx, USB Port 2 = 5xx) 1. Address straps are on the root sheet: port 1 ADCIN1 = LDO_3V3, ADCIN2 = GND (0x20); port 2 ADCIN1 = ADCIN2 = GND (0x21). R405-R408 are DNP divider footprints for other options. 2. Unused TPS25751 GPIOs tied to GND per datasheet (KiCad ERC flags this; expected). 3. At the connector pins: D402 CC ESD (24 V), D403 D+/D- ESD (5 V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"
- moved on the sheet: R412, R413, R414, R417, R421, R422, R423, R435

Commit message: Dev board: USB-C liquid detection, schematic review 3 fixes, new datasheets
Liquid detection (TPS25751 datasheet 9.2.2.2, both ports): TPD2S300 U405/U505
on SBU1/SBU2 into GPIO4/5, switched 100k pull-up / 1M pull-down (Q403-Q406)
on GPIO6/7. R440/R540 short D+/D- (passive BC1.2 DCP); D403/D503 removed.

Schematic review 3 (docs/devboard/schematic-review-3-2026-10-14.md):
- H1: TPD2S300 FLT -> GPIO3 fault input (SBU_FLT, R441 pull-up), as on
  TI's TPS25751EVM, so a VBUS-SBU short turns VBUS off.
- H2: R442/R443 hold the liquid-detect FETs off while GPIO6/7 are Hi-Z.
- H3: BQ25756 tuning parts from the EVM: 0R in gate and BTST lines
  (R444-R449), DNP RC snubbers on SW1/SW2 (R450/C454, R451/C455).
- H4: MonolithDev:TPS25751D, stock symbol with GPIO11 bidirectional;
  ERC now 0 errors, 8 expected GPIO-to-GND warnings.
- Gauge data flash and handling rules (Min Blow Fuse Voltage 10.5 V,
  COV Delay 1 s, no cell hot-swap with power on) in the bring-up
  checklist and gauge sheet note 15.
- Docs: A6 revision log, power budget, circuit description, README
  items 16/34/35/36.

Datasheets and app notes added (sources.csv): BQ2947, WSFB1514, TPD2S300,
BQ40Z50-R2 TRM, SLUA660, BQ25756 and TPS25751 EVM guides, discretes.

Co-Authored-By: Claude Opus 5.5 <noreply@anthropic.com>
Parts:
- removed D403: PESD5V0S2BT, Package_TO_SOT_SMD:SOT-23, symbol MonolithDev:ESD2CAN24
- added C451: 0.1u 50V, Capacitor_SMD:C_0603_1608Metric, symbol Device:C
- added C452, C453: 1u 50V, Capacitor_SMD:C_0603_1608Metric, symbol Device:C
- added C454, C455: 33p 50V, Capacitor_SMD:C_0603_1608Metric, symbol Device:C
- added Q403, Q404: AO3401A, Package_TO_SOT_SMD:SOT-23, symbol Transistor_FET:Q_PMOS_GSD
- added Q405, Q406: AO3400A, Package_TO_SOT_SMD:SOT-23, symbol Transistor_FET:Q_NMOS_GSD
- added R436, R437, R441, R442, R443: 100k, Resistor_SMD:R_0603_1608Metric, symbol Device:R
- added R438, R439: 1M, Resistor_SMD:R_0603_1608Metric, symbol Device:R
- added R440, R444, R445, R446, R447, R448, R449: 0R, Resistor_SMD:R_0603_1608Metric, symbol Device:R
- added R450, R451: 3.3R, Resistor_SMD:R_0805_2012Metric, symbol Device:R
- added U405: TPD2S300YFFR, MonolithDev:TI_YFF0009_DSBGA-9_P0.4mm, symbol MonolithDev:TPD2S300
- U401: symbol Interface_USB:TPS25751D -> MonolithDev:TPS25751D
Connections:
- net DN: now also R440.2; no longer U401.27 (GPIO5)
- net DP: now also R440.1; no longer U401.26 (GPIO4)
- net GND: now also C451.2, C452.2, C453.2, C454.2, C455.2, Q405.2 (S), Q406.2 (S), R443.2, U405.B2 (GND); no longer U401.19 (GPIO3), U401.36 (GPIO7), U401.37 (GPIO6)
- net HG1: now also R444.2; no longer U403.27 (HIDRV1)
- net HG2: now also R446.2; no longer U403.19 (HIDRV2)
- net LDO_3V3: now also C452.1, C453.1, Q403.2 (S), Q404.2 (S), R441.1, R442.1, U405.C2 (VPWR), U405.C3 (VM)
- net LG1: now also R445.2; no longer U403.25 (LODRV1)
- net LG2: now also R447.2; no longer U403.21 (LODRV2)
- net SW1: now also R450.1
- net SW2: now also R451.1
- net BTST2_C: now reaches C413.1, D405.1 (K)
- net BTST2_C: now also R449.2; no longer U403.20 (BTST2)
- net BTST1_C: now reaches C412.1, D404.1 (K)
- net BTST1_C: now also R448.2; no longer U403.26 (BTST1)
- net SBU1: now reaches J401.A8 (SBU1)
- net SBU1: now also U405.A1 (C_CC1)
- net SBU2: now reaches J401.B8 (SBU2)
- net SBU2: now also U405.A3 (C_CC2)
- new net: Q406.3 (D), R439.2
- new net: C454.1, R450.2
- new net: C455.1, R451.2
- new net: Q403.3 (D), R436.1
- new net: C451.1, U405.A2 (VBIAS)
- new net: Q404.3 (D), R437.1
- new net: Q405.3 (D), R438.2
- new net BTST1: R448.1, U403.26 (BTST1)
- new net BTST2: R449.1, U403.20 (BTST2)
- new net HIDRV1: R444.1, U403.27 (HIDRV1)
- new net HIDRV2: R446.1, U403.19 (HIDRV2)
- new net LIQ_PD: Q405.1 (G), Q406.1 (G), R443.1, U401.36 (GPIO7)
- new net LIQ_PU: Q403.1 (G), Q404.1 (G), R442.2, U401.37 (GPIO6)
- new net LODRV1: R445.1, U403.25 (LODRV1)
- new net LODRV2: R447.1, U403.21 (LODRV2)
- new net SBU1_SNS: R436.2, R438.1, U401.26 (GPIO4), U405.B1 (CC1)
- new net SBU2_SNS: R437.2, R439.1, U401.27 (GPIO5), U405.B3 (CC2)
- new net SBU_FLT: R441.2, U401.19 (GPIO3), U405.C1 (~{FLT})
- no-connect marks 3 -> 1
Other:
- note added: "GATE / BOOTSTRAP TUNING (BQ25756EVM fig. 3-1: R8, R20, R3, R17, R13, R23, snubbers)"
- note added: "LIQUID DETECTION (TPS25751 fig. 9-8)"
- note added: "NOTES (this sheet is used twice: USB Port 1 = 4xx, USB Port 2 = 5xx) 1. Address straps are on the root sheet: port 1 ADCIN1 = LDO_3V3, ADCIN2 = GND (0x20); port 2 ADCIN1 = ADCIN2 = GND (0x21). Both are SafeMode (TPS25751 table 8-6). 2. Unused TPS25751 GPIOs (0, 1, 2, 11) tied to GND per datasheet (KiCad ERC flags this; expected). Never configure them as outputs. 3. At the connector pins: D402 CC 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"
- note added: "USB-SIDE BULK: 4 x 22u MLCC + 100u polymer (>= 80 uF effective)"
- note removed: "NOTES (this sheet is used twice: USB Port 1 = 4xx, USB Port 2 = 5xx) 1. Address straps are on the root sheet: port 1 ADCIN1 = LDO_3V3, ADCIN2 = GND (0x20); port 2 ADCIN1 = ADCIN2 = GND (0x21). Both are SafeMode (TPS25751 table 8-6). 2. Unused TPS25751 GPIOs tied to GND per datasheet (KiCad ERC flags this; expected). 3. At the connector pins: D402 CC ESD (24 V), D403 D+/D- ESD (5 V: GPIO4/5 are ra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"
- note removed: "USB-SIDE BULK: 4 x 22u MLCC + 68u polymer (>= 80 uF effective)"

Commit message: Dev board: cost-down pass (about $113 -> $80 per board at 5 boards)
Swaps from docs/devboard/cost-down-2026-10-14.md, datasheet-checked:
- L401/L501 XAL7030 -> SMMS1040-2R2M (Isat 18 A, Irms 12 A, 9 mOhm)
- L402/L502 SRP5030T -> APS0530M3R3H (new footprint L_Coilank_APS0530)
- L201 SRN4018TA -> FNR4030S100MT
- U203 TPS70950 -> HT7550-1, C204/C205 10 uF per Holtek's basic circuit
- C431/C434/C435 47 uF 1210 -> 22 uF 1206 (bank ~114 uF effective)
- JLC basic/preferred equivalents: D103, D401, R410/R412, C105/C206,
  C406, Q103 -> AO3400A
- D301 (out of stock) -> red KT-0603R
- R431/R531 -> bridged solder jumper
- 34 test loops -> bare pads; pin headers hand-soldered
- U301 bought from ST and consigned to JLC

ERC unchanged (0 errors, 8 expected GPIO-to-GND warnings).

Co-Authored-By: Claude Opus 5.5 <noreply@anthropic.com>
Parts:
- C406: footprint Capacitor_SMD:C_0805_2012Metric -> Capacitor_SMD:C_1206_3216Metric; LCSC C20416422 -> C29823; MPN (none) -> 1206B475K500NT
- C431, C434, C435: value 47u 25V -> 22u 25V; footprint Capacitor_SMD:C_1210_3225Metric -> Capacitor_SMD:C_1206_3216Metric; LCSC C90142 -> C12891; MPN TMK325ABJ476MM-P -> CL31A226KAHNNNE; Notes (none) -> Battery-side ripple MLCC (cost-down 2026-10-14, was 47 uF 1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
- D401: LCSC C148220 -> C41376403; MPN (none) -> SMAJ22A (JLC preferred C41376403)
- J402: LCSC C2937625 -> (none); Sourcing (none) -> Hand-solder, not JLC assembled (through-hole; LCSC C2937625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
- L401: footprint Inductor_SMD:L_Coilcraft_XAL7030-222 -> Inductor_SMD:L_Changjiang_FXL1040; LCSC C19191686 -> C149591; MPN XAL7030-222MEC -> SMMS1040-2R2M (SXN); Notes (none) -> Cost-down 2026-10-14 (was Coilcraft XAL7030-222, $9.43): 2.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
- L402: footprint Inductor_SMD:L_Bourns_SRP5030T -> MonolithDev:L_Coilank_APS0530; LCSC C189931 -> C49073587; MPN SRP5030T-3R3M -> APS0530M3R3H (Coilank); Notes (none) -> Cost-down 2026-10-14 (was SRP5030T-3R3M): 3.3 uH, 38 mOhm m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
- R410, R412: footprint Resistor_SMD:R_0805_2012Metric -> Resistor_SMD:R_0603_1608Metric; LCSC C17678 -> C12447; MPN 0805W8F4022T5E -> 0603WAF4022T5E
- R431: value 0R -> Bridged; footprint Resistor_SMD:R_2512_6332Metric -> Jumper:SolderJumper-2_P1.3mm_Bridged2Bar_RoundedPad1.0x1.5mm; symbol Device:R -> Jumper:SolderJumper_2_Bridged; LCSC C2907567 -> (none); MPN FRC2512P000TS -> (none); Notes 2512 0R: carries up to ~1.7 A TPS62933 input (review m19) -> Cut both bars to isolate the TPS62933 input at bring-up (re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; now left out of the parts list
- TP401, TP402, TP403, TP404, TP407, TP408, TP409, TP410, TP411: footprint MonolithDev:TestPoint_Harwin_S2761_0603 -> TestPoint:TestPoint_Pad_D1.5mm; LCSC C55121754 -> (none); MPN RH-S2761-46R (ronghe; Harwin S2761-46R equivalent) -> (none); now left out of the parts list
Other:
- note added: "BATTERY-SIDE BULK: 3 x 22u MLCC + 100u polymer (>= 80 uF effective)"
- note removed: "BATTERY-SIDE BULK: 3 x 47u MLCC + 100u polymer (>= 80 uF effective)"
