File: DevBoard/mcu.kicad_sch (KiCad schematic)
At the start: 49 parts, among them J301 SWD, J302 UART debug, J303 Spare GPIO, SW301 RESET, U301 STM32WB1MMC

Commit message: Dev board rev A7: CC2340R5MODA MCU, TMP1075 sensors, shared IRQ_N
- U301 STM32WB1MMC -> TI CC2340R5MODA (cost-down; BLE only, on-chip OTA).
  New symbol and footprint (MHA0024A, with the fig. 9-2 antenna keep-out),
  RF match C313/R321/C314/C315, RSTN pull-up R302, wired per SWRS349A fig. 9-1.
- Only 10 usable GPIOs, so the five board NTCs become TMP1075 I2C sensors:
  U302-U304 fitted (port 1 stage, port 2 stage, connectors), U305/U306 DNP.
  FET over-temperature moves to the gauge internal sensor.
- TPS25751 IRQs, gauge BTP and TMP1075 ALERTs share one open-drain IRQ_N
  (R314 pull-up; R315, R114 DNP).
- R313 fitted at 470k: CC2340 pins float in reset, so it keeps the 3V3 rail
  out of sleep mode during boot.
- Pin budget doc, circuit description, bring-up checklist and README item 40
  updated; mcu-io-power-states.md flagged for rewrite. PCB not updated yet.

Co-Authored-By: Claude Opus 5.5 <noreply@anthropic.com>
Parts:
- removed R303: 0R, Resistor_SMD:R_0402_1005Metric, symbol Device:R
- removed R308, R309, R310, R311, R320: 10k 1%, Resistor_SMD:R_0805_2012Metric, symbol Device:R
- removed R316: 1k, Resistor_SMD:R_0603_1608Metric, symbol Device:R
- removed TH301, TH302, TH303, TH304, TH305: 10k B3435, Resistor_SMD:R_0603_1608Metric, symbol Device:Thermistor_NTC
- removed TP305: IRQ2, TestPoint:TestPoint_Pad_D1.5mm, symbol Connector:TestPoint
- removed TP306: BOOT0, TestPoint:TestPoint_Pad_D1.5mm, symbol Connector:TestPoint
- removed U301: STM32WB1MMC, MonolithDev:ST_LGA-77_STM32WB1MMC_6.5x10mm, symbol MonolithDev:STM32WB1MMC
- added C313: 15p C0G, Capacitor_SMD:C_0402_1005Metric, symbol Device:C
- added C314: TBD, Capacitor_SMD:C_0402_1005Metric, symbol Device:C
- added C315: 1p C0G, Capacitor_SMD:C_0402_1005Metric, symbol Device:C
- added R321: 0R, Resistor_SMD:R_0402_1005Metric, symbol Device:R
- added U301: CC2340R5MODA, MonolithDev:TI_MHA0024A_CC2340R5MODA_7x10mm, symbol MonolithDev:CC2340R5MODA
- added U302, U303, U304, U305, U306: TMP1075, Package_SON:Texas_DSG0008A_WSON-8-1EP_2x2mm_P0.5mm_EP0.9x1.6mm_ThermalVias, symbol Sensor_Temperature:TMP1075DSG
- C308, C309, C310: footprint Capacitor_SMD:C_0603_1608Metric -> Capacitor_SMD:C_0402_1005Metric; LCSC C14663 -> C307331; MPN CC0603KRX7R9BB104 -> CL05B104KB54PNC
- C311, C312: footprint Capacitor_SMD:C_0603_1608Metric -> Capacitor_SMD:C_0402_1005Metric; LCSC C14663 -> C307331; MPN CC0603KRX7R9BB104 -> CL05B104KB54PNC; now not fitted
- R302: value 10k -> 100k; LCSC C25804 -> C25803; MPN 0603WAF1002T5E -> 0603WAF1003T5E; Notes (none) -> TPS25751 I2Ct_IRQ is open drain and needs an external pull-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
- R313: value 100k -> 470k; LCSC C25803 -> (none); MPN 0603WAF1003T5E -> (none); now fitted
- R315: now not fitted
- TP304: value IRQ1 -> IRQ_N
Connections:
- net IRQ2 is gone; now on net IRQ_N: R315.2
- net NTC_TH1 is gone; now on net 3V3: C308.1
- net NTC_TH2 is gone; now on net 3V3: C309.1
- net NTC_TH3 is gone; now on net 3V3: C310.1
- net NTC_TH4 is gone; now on net 3V3: C311.1
- net 3V3: now also C312.1, U302.8 (V+), U303.7 (A0), U303.8 (V+), U304.6 (A1), U304.8 (V+), U305.6 (A1), U305.7 (A0), U305.8 (V+), U306.5 (A2), U306.8 (V+)
- net 3V3_MCU: now also R302.1, U301.6 (VDDS), U301.7 (VDDS)
- net 3V3_SLEEP: now also U301.15 (DIO21_A10)
- net CHG_INH: now also U301.11 (DIO24_A7)
- net EN_5V1: now also U301.12 (DIO3_X32P)
- net EN_5V2: now also U301.13 (DIO4_X32N)
- net GND: now also C314.2, C315.2, U301.1 (GND), U301.2 (GND), U301.22 (GND), U301.23 (GND), U301.24 (GND), U301.5 (GND), U301.8 (GND), U302.4 (GND), U302.5 (A2), U302.6 (A1), U302.7 (A0), U302.9 (EP), U303.4 (GND), U303.5 (A2), U303.6 (A1), U303.9 (EP), U304.4 (GND), U304.5 (A2), U304.7 (A0), U304.9 (EP), U305.4 (GND), U305.5 (A2), U305.9 (EP), U306.4 (GND), U306.6 (A1), U306.7 (A0), U306.9 (EP); no longer R302.2
- net LED_DRV: now also U301.18 (DIO12)
- net NRST: now also R302.2, U301.14 (RSTN)
- net SCL: now also U301.9 (DIO6_A1), U302.2 (SCL), U303.2 (SCL), U304.2 (SCL), U305.2 (SCL), U306.2 (SCL)
- net SDA: now also U301.10 (DIO8), U302.1 (SDA), U303.1 (SDA), U304.1 (SDA), U305.1 (SDA), U306.1 (SDA)
- net UART_RX: now also U301.17 (DIO20_A11)
- net UART_TX: now also U301.16 (DIO18)
- net at J301.2 (Pin_2): now also U301.20 (DIO16/SWDIO)
- net at J301.4 (Pin_4): now also U301.19 (DIO17/SWDCK)
- net IRQ1 renamed IRQ_N
- net IRQ_N: now also J303.2 (Pin_2), U301.21 (DIO11), U302.3 (ALERT), U303.3 (ALERT), U304.3 (ALERT), U305.3 (ALERT), U306.3 (ALERT)
- net J303_NTC_EN: no longer names the net of J303.3 (Pin_3)
- removed net NTC_TH5: C312.1, J303.2 (Pin_2)
- new net: C313.2, C314.1, R321.1
- new net ANT_IN: C315.1, R321.2, U301.3 (ANT_IN)
- new net RFIO: C313.1, U301.4 (RFIO)
- no-connect marks 6 -> 4
Other:
- note added: "0x48: port 1 stage (TH301)"
- note added: "0x49: port 2 stage (TH302)"
- note added: "0x4A: USB-C connectors (TH303)"
- note added: "0x4B: DNP, heatsink (TH304)"
- note added: "0x4C: DNP, prot. FETs (TH305)"
- note added: "BLUETOOTH MCU CC2340R5MODA (per TI SWRS349A fig. 9-1)"
- note added: "BOARD TEMPERATURE (TMP1075 on I2C, 0x48-0x4C; ALERT wire-ORed onto IRQ_N)"
- note added: "NOTES 1. U301 antenna end at a board edge, ground 10-20 mm each side; keep-out in the footprint (fig. 9-2). 2. C301-C303 at the VDDS pads. R302 + C304 = power-on reset (SWRS349A fig. 9-1 R1/C92). 3. C313 = CA1. R321/C314/C315 = Z61/Z60/Z62 pi match (TI: 0R, DNP, 1 pF); retune on the board. 4. No 32 kHz crystal: LFOSC calibrated against the 48 MHz crystal. DIO3/DIO4 are GPIOs. 5. Pins: DIO6 SCL, D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"
- note removed: "BLUETOOTH MCU STM32WB1MMC (per ST DS14096 fig. 5)"
- note removed: "BOARD NTCs (TH1-TH4, divider powered only while sampling)"
- note removed: "NOTES 1. U301 at a board edge, as on ST's reference PCB (DS14096 fig. 6): copper-free notch past the antenna end. 2. C301-C303 at the VDD pads; C304 at NRST. 3. PB0/PB1/PB2 left unconnected (ST: RF-sensitive pins). NTC_EN = PA8, EN_5V1 = PA11, EN_5V2 = PA12. 4. R303 0R joins ANT_IN/ANT_OUT for the internal antenna (ST fig. 2). 5. Pin map checked against DS13258 table 15: NTC ADC1_IN6/8/9/10 (+ IN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"
- title: MCU and board NTCs -> MCU and board temperature

Commit message: Dev board rev A7 layout: CC2340R5MODA and TMP1075 placed
- Board updated to the rev A7 schematic: U301 CC2340R5MODA at the top edge
  with its RF match, TMP1075 U302-U306 on the copper they measure.
- TMP1075 footprint with 0.3 mm thermal vias (JLC minimum) in place of
  KiCad's 0.2 mm ThermalVias variant.
- DRC 0 errors, schematic parity 0, ERC at the usual 8 warnings.

Co-Authored-By: Claude Opus 5.5 <noreply@anthropic.com>
Parts:
- U302, U303, U304, U305, U306: footprint Package_SON:Texas_DSG0008A_WSON-8-1EP_2x2mm_P0.5mm_EP0.9x1.6mm_ThermalVias -> MonolithDev:TI_DSG0008A_WSON-8-1EP_2x2mm_P0.5mm_EP0.9x1.6mm_Vias0.3mm
Changed lines of the file:
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@@
 			)
 		)
-		(property "Footprint" "Package_SON:Texas_DSG0008A_WSON-8-1EP_2x2mm_P0.5mm_EP0.9x1.6mm_ThermalVias"
+		(property "Footprint" "MonolithDev:TI_DSG0008A_WSON-8-1EP_2x2mm_P0.5mm_EP0.9x1.6mm_Vias0.3mm"
 			(at 60.96 200.66 0)
 			(hide yes)
@@
 			)
 		)
-		(property "Footprint" "Package_SON:Texas_DSG0008A_WSON-8-1EP_2x2mm_P0.5mm_EP0.9x1.6mm_ThermalVias"
+		(property "Footprint" "MonolithDev:TI_DSG0008A_WSON-8-1EP_2x2mm_P0.5mm_EP0.9x1.6mm_Vias0.3mm"
 			(at 101.6 200.66 0)
 			(hide yes)
@@
 			)
 		)
-		(property "Footprint" "Package_SON:Texas_DSG0008A_WSON-8-1EP_2x2mm_P0.5mm_EP0.9x1.6mm_ThermalVias"
+		(property "Footprint" "MonolithDev:TI_DSG0008A_WSON-8-1EP_2x2mm_P0.5mm_EP0.9x1.6mm_Vias0.3mm"
 			(at 142.24 200.66 0)
 			(hide yes)
@@
 			)
 		)
-		(property "Footprint" "Package_SON:Texas_DSG0008A_WSON-8-1EP_2x2mm_P0.5mm_EP0.9x1.6mm_ThermalVias"
+		(property "Footprint" "MonolithDev:TI_DSG0008A_WSON-8-1EP_2x2mm_P0.5mm_EP0.9x1.6mm_Vias0.3mm"
 			(at 124.46 241.3 0)
 			(hide yes)
@@
 			)
 		)
-		(property "Footprint" "Package_SON:Texas_DSG0008A_WSON-8-1EP_2x2mm_P0.5mm_EP0.9x1.6mm_ThermalVias"
+		(property "Footprint" "MonolithDev:TI_DSG0008A_WSON-8-1EP_2x2mm_P0.5mm_EP0.9x1.6mm_Vias0.3mm"
 			(at 165.1 241.3 0)
 			(hide yes)
