File: DevBoard/mcu.kicad_sch (KiCad schematic)
At the start: 47 parts, among them J301 SWD, J302 UART debug, J303 Spare GPIO, SW301 RESET, U301 CC2340R5MODA, U302 TMP1075, U303 TMP1075, U304 TMP1075, U305 TMP1075, U306 TMP1075

Commit message: Layout in progress
Backup before replicate
Parts:
- TP309: footprint MonolithDev:TestPoint_Harwin_S2761_0603 -> TestPoint:TestPoint_Pad_D1.5mm
