File: DevBoard/mcu.kicad_sch (KiCad schematic)
At the start: 47 parts, among them J301 SWD, J302 UART debug, J303 Spare GPIO, SW301 RESET, U301 CC2340R5MODA, U302 TMP1075, U303 TMP1075, U304 TMP1075, U305 TMP1075, U306 TMP1075

Commit message: Dev board: 10R gate resistors with turn-off diodes; remove TMP1075 sensors
Gate drive (both ports): R444-R447 / R544-R547 0R -> 10R, with a BAT54WS
(D406-D409 / D506-D509) across each, cathode at the BQ25756 driver pin, so
turn-off bypasses the resistor and the 45 ns dead time is kept. Notes on the
gate resistors rewritten (they named the wrong drivers). Diodes are staged
below the board for hand placement.

Board temperature (rev A8): U302-U306 and C308-C312 removed. Temperatures
now come from the gauge (DAStatus2: TS1-TS4, cell, FET, die; readable
sealed) and from each BQ25756 TS NTC via the TPS25751 'I2Cr' pass-through
(REG0x37 TS_ADC). IRQ_N now has three sources. Docs, power budget and
scripts updated.

Also includes the author's own uncommitted schematic and README edits.
ERC: 8 known warnings; DRC schematic parity: 0 footprint errors.

Co-Authored-By: Claude Opus 5.5 <noreply@anthropic.com>
Parts:
- removed C308, C309, C310, C311, C312: 0.1u 50V, Capacitor_SMD:C_0402_1005Metric, symbol Device:C
- removed U302, U303, U304, U305, U306: TMP1075, MonolithDev:TI_DSG0008A_WSON-8-1EP_2x2mm_P0.5mm_EP0.9x1.6mm_Vias0.3mm, symbol Sensor_Temperature:TMP1075DSG
- R314: Notes The one IRQ_N pull-up (TPS25751 I2Ct_IRQ x2, gauge BTP via Q103, TMP1075 ALERTs; all open drain). 47k for leakage and noise margin on a long net (review 4 A-5); 70 uA only while asserted -> The one IRQ_N pull-up (TPS25751 I2Ct_IRQ x2, gauge BTP via Q103; all open drain). 47k for leakage and noise margin on a long net (review 4 A-5); 70 uA only while asserted
Other:
- note removed: "0x48: port 1 stage (TH301)"
- note removed: "0x49: port 2 stage (TH302)"
- note removed: "0x4A: USB-C connectors (TH303)"
- note removed: "0x4B: DNP, heatsink (TH304)"
- note removed: "0x4C: DNP, prot. FETs (TH305)"
- note removed: "BOARD TEMPERATURE (TMP1075 on I2C, 0x48-0x4C; ALERT wire-ORed onto IRQ_N)"
