File: DevBoard/gauge.kicad_sch (KiCad schematic)
At the start: 79 parts, among them J101 Pack (welded 4S) - use instea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, J102 Cell 1 NTC 10k 103AT, J103 EV2400 SMBus, J104 Bench PACK_P, J105 Cell 2 NTC 10k 103AT, J106 Cell 3 NTC 10k 103AT, J107 Cell 4 NTC 10k 103AT, Q101 AGM404AP1, Q102 AGM404AP1, Q103 AO3400A, Q104 AO3400A, SW101 WAKE, U101 BQ40Z50RSMR-R2, U102 BQ294700DSGR

Commit message: Layout in progress
Backup before replicate
Parts:
- TP109: footprint MonolithDev:TestPoint_Harwin_S2761_0603 -> TestPoint:TestPoint_Pad_D1.5mm
