File: DevBoard/power.kicad_sch (KiCad schematic)
At the start: 31 parts, among them U201 INA190A5IDDFR, U202 INA190A1IDDFR, U203 HT7550-1, U204 TPS62177DQCR

Commit message: Layout in progress
Backup before replicate
Parts:
- TP201, TP202, TP203, TP208, TP209: footprint MonolithDev:TestPoint_Harwin_S2761_0603 -> TestPoint:TestPoint_Pad_D1.5mm
Changed lines of the file:
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@@
 	(wire
 		(pts
-			(xy 68.58 229.87) (xy 80.01 229.87)
+			(xy 68.58 229.87) (xy 81.28 229.87)
 		)
 		(stroke
@@
 	(wire
 		(pts
-			(xy 97.79 229.87) (xy 106.68 229.87)
-		)
-		(stroke
-			(width 0)
-			(type default)
-		)
-	)
-	(wire
-		(pts
 			(xy 121.92 59.69) (xy 121.92 55.88)
 		)
@@
 	(wire
 		(pts
+			(xy 96.52 229.87) (xy 106.68 229.87)
+		)
+		(stroke
+			(width 0)
+			(type default)
+		)
+	)
+	(wire
+		(pts
 			(xy 143.51 144.78) (xy 152.4 144.78)
 		)
@@
 			)
 		)
-		(property "Footprint" "MonolithDev:TestPoint_Harwin_S2761_0603"
+		(property "Footprint" "TestPoint:TestPoint_Pad_D1.5mm"
 			(at 195.58 165.1 0)
 			(hide yes)
@@
 			)
 		)
-		(property "Notes" "HT7550 input: Holtek basic circuit 10 uF; 50 V and more C damp the JP202 hot-plug ring"
+		(property "Description" "Unpolarized capacitor"
 			(at 68.58 233.68 0)
 			(hide yes)
@@
 			)
 		)
-		(property "Description" "Unpolarized capacitor"
+		(property "Notes" "HT7550 input: Holtek basic circuit 10 uF; 50 V and more C damp the JP202 hot-plug ring"
 			(at 68.58 233.68 0)
 			(hide yes)
@@
 			)
 		)
-		(property "Footprint" "MonolithDev:TestPoint_Harwin_S2761_0603"
+		(property "Footprint" "TestPoint:TestPoint_Pad_D1.5mm"
 			(at 157.48 144.78 0)
 			(hide yes)
@@
 			)
 		)
-		(property "Sourcing" "Hand-solder, not JLC assembled (through-hole; LCSC C492401 PZ254V-11-02P)"
+		(property "Description" "Jumper, 2-pole, open"
 			(at 50.8 229.87 0)
 			(hide yes)
@@
 			)
 		)
-		(property "Description" "Jumper, 2-pole, open"
+		(property "Sourcing" "Hand-solder, not JLC assembled (through-hole; LCSC C492401 PZ254V-11-02P)"
 			(at 50.8 229.87 0)
 			(hide yes)
@@
 	(symbol
 		(lib_id "Regulator_Linear:HT75xx-1-SOT89")
-		(at 88.90 232.41 0)
+		(at 88.9 232.41 0)
 		(unit 1)
 		(body_style 1)
@@
 			)
 		)
-		(property "Notes" "Cost-down 2026-10-14 (was TPS70950DBVR): JLC preferred. Supplies only the two INA190s. +/-3 %, 30 V max input: the JP202 hot-plug ring (review 2 C-3, 23-30 V) is why C204 is 10 uF 50 V. Holtek basic circuit: 10 uF in and out. No EN pin (the TPS709 EN was left open)"
+		(property "Description" "Holtek HT7550-1 5 V LDO, 30 V input, 2.5 uA Iq, SOT-89 (1 GND, 2 VIN, 3 VOUT)"
 			(at 88.9 231.14 0)
 			(hide yes)
@@
 			)
 		)
-		(property "MPN" "HT7550-1 (Holtek)"
+		(property "Notes" "Cost-down 2026-10-14 (was TPS70950DBVR): JLC preferred. Supplies only the two INA190s. +/-3 %, 30 V max input: the JP202 hot-plug ring (review 2 C-3, 23-30 V) is why C204 is 10 uF 50 V. Holtek basic circuit: 10 uF in and out. No EN pin (the TPS709 EN was left open)"
 			(at 88.9 231.14 0)
 			(hide yes)
@@
 			)
 		)
-		(property "Description" "Holtek HT7550-1 5 V LDO, 30 V input, 2.5 uA Iq, SOT-89 (1 GND, 2 VIN, 3 VOUT)"
+		(property "MPN" "HT7550-1 (Holtek)"
 			(at 88.9 231.14 0)
 			(hide yes)
@@
 			)
 		)
-		(property "Footprint" "MonolithDev:TestPoint_Harwin_S2761_0603"
+		(property "Footprint" "TestPoint:TestPoint_Pad_D1.5mm"
 			(at 177.8 152.4 0)
 			(hide yes)
@@
 			)
 		)
-		(property "Sourcing" "Hand-solder, not JLC assembled (through-hole; LCSC C492401 PZ254V-11-02P)"
+		(property "Description" "Jumper, 2-pole, open"
 			(at 132.08 229.87 0)
 			(hide yes)
@@
 			)
 		)
-		(property "Description" "Jumper, 2-pole, open"
+		(property "Sourcing" "Hand-solder, not JLC assembled (through-hole; LCSC C492401 PZ254V-11-02P)"
 			(at 132.08 229.87 0)
 			(hide yes)
@@
 			)
 		)
-		(property "Notes" "10 uH as in the TPS62177 datasheet application (LPS4018-103); 130 mOhm, 1.6 A Irms / 2.4 A Isat for a 0.5 A converter. Cost-down 2026-10-14 (was SRN4018TA-100M)"
+		(property "Description" "Inductor"
 			(at 175.26 55.88 0)
 			(hide yes)
@@
 			)
 		)
-		(property "Description" "Inductor"
+		(property "Notes" "10 uH as in the TPS62177 datasheet application (LPS4018-103); 130 mOhm, 1.6 A Irms / 2.4 A Isat for a 0.5 A converter. Cost-down 2026-10-14 (was SRN4018TA-100M)"
 			(at 175.26 55.88 0)
 			(hide yes)
@@
 			)
 		)
-		(property "Footprint" "MonolithDev:TestPoint_Harwin_S2761_0603"
+		(property "Footprint" "TestPoint:TestPoint_Pad_D1.5mm"
 			(at 177.8 190.5 0)
 			(hide yes)
@@
 			)
 		)
-		(property "Footprint" "MonolithDev:TestPoint_Harwin_S2761_0603"
+		(property "Footprint" "TestPoint:TestPoint_Pad_D1.5mm"
 			(at 157.48 182.88 0)
 			(hide yes)
@@
 		)
 	)
-	(wire
-		(pts
-			(xy 80.01 229.87) (xy 81.28 229.87)
-		)
-		(stroke
-			(width 0)
-			(type default)
-		)
-	)
-	(wire
-		(pts
-			(xy 96.52 229.87) (xy 97.79 229.87)
-		)
-		(stroke
-			(width 0)
-			(type default)
-		)
-	)
