File: Production/gauge.kicad_sch (KiCad schematic)
At the start: 65 parts, among them J102 Cell 1 NTC wires, J105 Cell 2 NTC wires, J106 Cell 3 NTC wires, J107 Cell 4 NTC wires, J108 PACK- (CELL_N), J109 CELL1 tap, J110 CELL2 tap, J111 CELL3 tap, J112 PACK+ (CELL_P_RAW), Q101 AGM404AP1, Q102 AGM404AP1, Q103 AO3400A, Q104 AO3400A, U101 BQ40Z50RSMR-R2, U102 BQ294700DSGR

Commit message: Production schematic P0: drawing tidy
tools/tidy_production.py (runs after make_production.py): pogo pads in their
own row, TC2030 under its SWD heading, link-merge leftovers removed, empty
headings deleted, sheet notes, root index and revision log rewritten for
production, sheets renamed 3V3 Rail and MCU. Netlist unchanged (check_netlist
passes); ERC: no errors.

Co-Authored-By: Claude Opus 5.5 <noreply@anthropic.com>
Other:
- note added: "FACTORY TEST PADS"
- note added: "GAUGE SMBus (0x0B) + POGO PADS"
- note added: "J108 PACK- and J112 PACK+: 16 AWG leads in 1.7 mm plated holes. J109-J111: cell tap wires. Connect with USB unplugged, in order: PACK-, CELL1, CELL2, CELL3, PACK+ (note 15)."
- note added: "NOTES 1. CELL_N = gauge VSS (cell 1 negative). GND = system ground, on the far side of RS101. 2. Kelvin-route SRP/SRN from the RS101 pads; R107/R108/C106 at the IC. 3. VC taps are separate thin traces from the tap pads J109-J111 and from the J108/J112 pads; VC4 from CELL_P_RAW (before F102) so fuse drop is not read as cell voltage. 4. TS1-TS4: one wired 10k NTC per cell on J102, J105-J107, taped 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"
- note added: "PACK WIRES (welded 4S EVE INR21700-58E)"
- note removed: "CELL STACK (4S)"
- note removed: "HOST SMBus (gauge 0x0B) / EV2400"
- note removed: "Holders BT101-BT104 OR welded pack on J101 - never both. J101 is DNP. Check each cell at TP102-TP105 and the stack at TP108 before waking the gauge (Q101/Q102 stay off until FET_EN is set, so nothing loads the cells until then)."
- note removed: "NOTES 1. CELL_N = gauge VSS (cell 1N tab). GND = system ground, on the far side of RS101. 2. Kelvin-route SRP/SRN from the RS101 pads; R107/R108/C106 at the IC. 3. VC taps are separate thin traces from the cell end of each holder contact; VC4 from CELL_P_RAW (before F102) so fuse drop is not read as cell voltage. 4. TS1-TS4: one wired cell NTC each (J102, J105-J107, one per cell); insulated senso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"
- note removed: "TEST POINTS / POWER FLAGS"
- note removed: "WAKE + BENCH SUPPLY"

Commit message: Production schematic P0: passive downsizing (-432 mm2 courtyard, -16 %)
Extended parts and 0201 allowed on production (0201 only where both nets stay
<= 5.5 V). Charger inductor 10x10 -> Coilank APS0730M2R2F; 0603 R -> 0402;
low-voltage R/C -> 0201; RAC 0805, RBAT 1206, gauge shunt 1206; R101-R104
0402; BAT54 SOD-882; REGN/filter/SS caps 0402; NTC 0402. Bulk polymers and
TPS25751/TPS62933 caps kept (leakage, derating). New APS0730 footprint is
written by make_production.py. Netlist check passes; ERC clean.

Co-Authored-By: Claude Opus 5.5 <noreply@anthropic.com>
Parts:
- D101: footprint Diode_SMD:D_SOD-323 -> Diode_SMD:D_SOD-882; LCSC C7502694 -> C549279; MPN BAT54WS (R+O) -> BAT54L,315 (Nexperia)
- R101, R102, R103, R104: footprint Resistor_SMD:R_1206_3216Metric -> Resistor_SMD:R_0402_1005Metric; LCSC C17901 -> C25076; MPN 1206W4F1000T5E -> 0402WGF1000TCE
- R110, R112: value 10M -> 10M 5%; footprint Resistor_SMD:R_0603_1608Metric -> Resistor_SMD:R_0402_1005Metric; LCSC C7250 -> C26086; MPN 0603WAF1005T5E -> 0402WGJ0106TCE
- R115, R116: footprint Resistor_SMD:R_0402_1005Metric -> Resistor_SMD:R_0201_0603Metric; LCSC C25076 -> C270366; MPN 0402WGF1000TCE -> 0201WMF1000TEE
- R117: footprint Resistor_SMD:R_0603_1608Metric -> Resistor_SMD:R_0402_1005Metric; LCSC C23178 -> C25790; MPN 0603WAF4703T5E -> 0402WGF4703TCE
- RS101: value 1m 1% 2W -> 1m 1% 1W; footprint Resistor_SMD:R_2512_6332Metric -> Resistor_SMD:R_1206_3216Metric; LCSC C326570 -> C154629; MPN PA2512FKE7W0R001E -> LR1206-21R001F4 (Ralec, 75 ppm)
Other:
- note added: "NOTES 1. CELL_N = gauge VSS (cell 1 negative). GND = system ground, on the far side of RS101. 2. Kelvin-route SRP/SRN from the RS101 pads; R107/R108/C106 at the IC. RS101 is a 1206 1 W 75 ppm alloy part (P0). 3. VC taps are separate thin traces from the tap pads J109-J111 and from the J108/J112 pads; VC4 from CELL_P_RAW (before F102) so fuse drop is not read as cell voltage. 4. TS1-TS4: one wired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"
- note removed: "NOTES 1. CELL_N = gauge VSS (cell 1 negative). GND = system ground, on the far side of RS101. 2. Kelvin-route SRP/SRN from the RS101 pads; R107/R108/C106 at the IC. 3. VC taps are separate thin traces from the tap pads J109-J111 and from the J108/J112 pads; VC4 from CELL_P_RAW (before F102) so fuse drop is not read as cell voltage. 4. TS1-TS4: one wired 10k NTC per cell on J102, J105-J107, taped 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"
Changed lines of the file:
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@@
 		)
 	)
-	(text "NOTES\n1. CELL_N = gauge VSS (cell 1 negative). GND = system ground, on the far side of RS101.\n2. Kelvin-route SRP/SRN from the RS101 pads; R107/R108/C106 at the IC.\n3. VC taps are separate thin traces from the tap pads J109-J111 and from the J108/J112 pads;\n    VC4 from CELL_P_RAW (before F102) so fuse drop is not read as cell voltage.\n4. TS1-TS4: one wired 10k NTC per cell on J102, J105-J107, taped to the cell at mid-height; insulated sensors only\n    (cans 0-12.6 V above VSS, TS 2.1 V max). PTC, PTCEN, PRES, DISP tied to VSS per datasheet.\n5. VCC fed from FET common drain via R106 (TI R13). PACK sense via R113 10k (TI R15).\n6. BAT fed from CELL_P_RAW (cell top, before F102) via D101 + R105 (TI fig. 9-12).\n7. Diamonds are PWR_FLAGs (ERC only, no part): each sits where its rail is sourced through a passive part.\n8. Q103 buffers BTP_INT onto the shared open-drain IRQ_N (CC2340 DIO11): IRQ_N is low while BTP_INT is high.\n   Keep BTP disabled, or set BTP_POL = 1 with BTP_EN = 1, or IRQ_N is held low (review 4 D-2).\n9. D103 clamps Q102 VGS at 15 V in a hard short. The dev board's C109/D102 inrush options are not on P0.\n10. No wake button: the gauge leaves SHUTDOWN when PACK_P comes up, i.e. when USB is plugged in (TPS25751 dead-battery\n    sink + BQ25756 charging with 3V3 down, USB sheet note 11). Confirm on the dev board.\n11. TP110-TP112 = SMBus pogo pads (SMBC, SMBD, GND) for an EV2400 / BQStudio: golden image and calibration.\n    Only with 3V3 up and U301 held in reset (MCU sheet note 10).\n12. TP106 PACK_P and TP109 GND are factory test pads.\n13. ESD caps (TI): C110+C111 in series across the FET pair (fig. 9-2 C1/C2), C107+C108 across PACK+/PACK- (sec. 9.2.2.1.5).\n14. Second level (TI fig. 9-11): U102 BQ294700 (4.35 V/cell, CD 0.1u = 1-2 s) or the gauge FUSE pin turns Q104 on;\n    F102's heater then blows its fuse, permanently opening the cell top. F102 is also the pack's only overcurrent fuse.\n15. Connect the pack with USB unplugged, PACK- first, then the taps bottom-up, then PACK+: a floating tap can read\n    > 4.35 V, U102 trips after 1-2 s and F102 blows. Gauge data flash: COV Delay 1 s, Min Blow Fuse Voltage 10500 mV."
+	(text "NOTES\n1. CELL_N = gauge VSS (cell 1 negative). GND = system ground, on the far side of RS101.\n2. Kelvin-route SRP/SRN from the RS101 pads; R107/R108/C106 at the IC. RS101 is a 1206 1 W 75 ppm alloy part (P0).\n3. VC taps are separate thin traces from the tap pads J109-J111 and from the J108/J112 pads;\n    VC4 from CELL_P_RAW (before F102) so fuse drop is not read as cell voltage.\n4. TS1-TS4: one wired 10k NTC per cell on J102, J105-J107, taped to the cell at mid-height; insulated sensors only\n    (cans 0-12.6 V above VSS, TS 2.1 V max). PTC, PTCEN, PRES, DISP tied to VSS per datasheet.\n5. VCC fed from FET common drain via R106 (TI R13). PACK sense via R113 10k (TI R15).\n6. BAT fed from CELL_P_RAW (cell top, before F102) via D101 + R105 (TI fig. 9-12).\n7. Diamonds are PWR_FLAGs (ERC only, no part): each sits where its rail is sourced through a passive part.\n8. Q103 buffers BTP_INT onto the shared open-drain IRQ_N (CC2340 DIO11): IRQ_N is low while BTP_INT is high.\n   Keep BTP disabled, or set BTP_POL = 1 with BTP_EN = 1, or IRQ_N is held low (review 4 D-2).\n9. D103 clamps Q102 VGS at 15 V in a hard short. The dev board's C109/D102 inrush options are not on P0.\n10. No wake button: the gauge leaves SHUTDOWN when PACK_P comes up, i.e. when USB is plugged in (TPS25751 dead-battery\n    sink + BQ25756 charging with 3V3 down, USB sheet note 11). Confirm on the dev board.\n11. TP110-TP112 = SMBus pogo pads (SMBC, SMBD, GND) for an EV2400 / BQStudio: golden image and calibration.\n    Only with 3V3 up and U301 held in reset (MCU sheet note 10).\n12. TP106 PACK_P and TP109 GND are factory test pads.\n13. ESD caps (TI): C110+C111 in series across the FET pair (fig. 9-2 C1/C2), C107+C108 across PACK+/PACK- (sec. 9.2.2.1.5).\n14. Second level (TI fig. 9-11): U102 BQ294700 (4.35 V/cell, CD 0.1u = 1-2 s) or the gauge FUSE pin turns Q104 on;\n    F102's heater then blows its fuse, permanently opening the cell top. F102 is also the pack's only overcurrent fuse.\n15. Connect the pack with USB unplugged, PACK- first, then the taps bottom-up, then PACK+: a floating tap can read\n    > 4.35 V, U102 trips after 1-2 s and F102 blows. Gauge data flash: COV Delay 1 s, Min Blow Fuse Voltage 10500 mV."
 		(exclude_from_sim no)
 		(at 196.596 248.412 0)
@@
 			)
 		)
-		(property "Footprint" "Resistor_SMD:R_0402_1005Metric"
+		(property "Footprint" "Resistor_SMD:R_0201_0603Metric"
 			(at 257.81 152.908 90)
 			(hide yes)
@@
 			)
 		)
-		(property "LCSC" "C25076"
+		(property "LCSC" "C270366"
 			(at 257.81 151.13 0)
 			(hide yes)
@@
 			)
 		)
-		(property "MPN" "0402WGF1000TCE"
+		(property "MPN" "0201WMF1000TEE"
 			(at 257.81 151.13 0)
 			(hide yes)
@@
 			)
 		)
-		(property "Footprint" "Resistor_SMD:R_1206_3216Metric"
+		(property "Footprint" "Resistor_SMD:R_0402_1005Metric"
 			(at 160.02 149.098 90)
 			(hide yes)
@@
 			)
 		)
-		(property "LCSC" "C17901"
+		(property "LCSC" "C25076"
 			(at 160.02 147.32 0)
 			(hide yes)
@@
 			)
 		)
-		(property "MPN" "1206W4F1000T5E"
+		(property "MPN" "0402WGF1000TCE"
 			(at 160.02 147.32 0)
 			(hide yes)
@@
 			)
 		)
-		(property "Value" "10M"
+		(property "Value" "10M 5%"
 			(at 166.79 61.79 0)
 			(show_name no)
@@
 			)
 		)
-		(property "Footprint" "Resistor_SMD:R_0603_1608Metric"
+		(property "Footprint" "Resistor_SMD:R_0402_1005Metric"
 			(at 160.782 60.96 90)
 			(hide yes)
@@
 			)
 		)
-		(property "LCSC" "C7250"
+		(property "LCSC" "C26086"
 			(at 162.56 60.96 0)
 			(hide yes)
@@
 			)
 		)
-		(property "MPN" "0603WAF1005T5E"
+		(property "MPN" "0402WGJ0106TCE"
 			(at 162.56 60.96 0)
 			(hide yes)
@@
 			)
 		)
-		(property "Footprint" "Resistor_SMD:R_0402_1005Metric"
+		(property "Footprint" "Resistor_SMD:R_0201_0603Metric"
 			(at 240.03 150.368 90)
 			(hide yes)
@@
 			)
 		)
-		(property "LCSC" "C25076"
+		(property "LCSC" "C270366"
 			(at 240.03 148.59 0)
 			(hide yes)
@@
 			)
 		)
-		(property "MPN" "0402WGF1000TCE"
+		(property "MPN" "0201WMF1000TEE"
 			(at 240.03 148.59 0)
 			(hide yes)
@@
 			)
 		)
-		(property "Footprint" "Resistor_SMD:R_1206_3216Metric"
+		(property "Footprint" "Resistor_SMD:R_0402_1005Metric"
 			(at 160.02 171.958 90)
 			(hide yes)
@@
 			)
 		)
-		(property "LCSC" "C17901"
+		(property "LCSC" "C25076"
 			(at 160.02 170.18 0)
 			(hide yes)
@@
 			)
 		)
-		(property "MPN" "1206W4F1000T5E"
+		(property "MPN" "0402WGF1000TCE"
 			(at 160.02 170.18 0)
 			(hide yes)
@@
 			)
 		)
-		(property "Footprint" "Diode_SMD:D_SOD-323"
+		(property "Footprint" "Diode_SMD:D_SOD-882"
 			(at 179.07 135.89 0)
 			(hide yes)
@@
 			)
 		)
-		(property "LCSC" "C7502694"
+		(property "LCSC" "C549279"
 			(at 179.07 135.89 0)
 			(hide yes)
@@
 			)
 		)
-		(property "MPN" "BAT54WS (R+O)"
+		(property "MPN" "BAT54L,315 (Nexperia)"
 			(at 179.07 135.89 0)
 			(hide yes)
@@
 			)
 		)
-		(property "Footprint" "Resistor_SMD:R_1206_3216Metric"
+		(property "Footprint" "Resistor_SMD:R_0402_1005Metric"
 			(at 160.02 164.338 90)
 			(hide yes)
@@
 			)
 		)
-		(property "LCSC" "C17901"
+		(property "LCSC" "C25076"
 			(at 160.02 162.56 0)
 			(hide yes)
@@
 			)
 		)
-		(property "MPN" "1206W4F1000T5E"
+		(property "MPN" "0402WGF1000TCE"
 			(at 160.02 162.56 0)
 			(hide yes)
@@
 			)
 		)
-		(property "Footprint" "Resistor_SMD:R_1206_3216Metric"
+		(property "Footprint" "Resistor_SMD:R_0402_1005Metric"
 			(at 160.02 156.718 90)
 			(hide yes)
@@
 			)
 		)
-		(property "LCSC" "C17901"
+		(property "LCSC" "C25076"
 			(at 160.02 154.94 0)
 			(hide yes)
@@
 			)
 		)
-		(property "MPN" "1206W4F1000T5E"
+		(property "MPN" "0402WGF1000TCE"
 			(at 160.02 154.94 0)
 			(hide yes)
@@
 			)
 		)
-		(property "Value" "1m 1% 2W"
+		(property "Value" "1m 1% 1W"
 			(at 63.35 218.18 90)
 			(show_name no)
@@
 			)
 		)
-		(property "Footprint" "Resistor_SMD:R_2512_6332Metric"
+		(property "Footprint" "Resistor_SMD:R_1206_3216Metric"
 			(at 63.5 222.758 90)
 			(hide yes)
@@
 			)
 		)
-		(property "LCSC" "C326570"
+		(property "LCSC" "C154629"
 			(at 63.5 220.98 0)
 			(hide yes)
@@
 			)
 		)
-		(property "MPN" "PA2512FKE7W0R001E"
+		(property "MPN" "LR1206-21R001F4 (Ralec, 75 ppm)"
 			(at 63.5 220.98 0)
 			(hide yes)
@@
 			)
 		)
-		(property "Footprint" "Resistor_SMD:R_0603_1608Metric"
+		(property "Footprint" "Resistor_SMD:R_0402_1005Metric"
 			(at 332.74 190.5 0)
 			(hide yes)
@@
 			)
 		)
-		(property "LCSC" "C23178"
+		(property "LCSC" "C25790"
 			(at 332.74 190.5 0)
 			(hide yes)
@@
 			)
 		)
-		(property "MPN" "0603WAF4703T5E"
+		(property "MPN" "0402WGF4703TCE"
 			(at 332.74 190.5 0)
 			(hide yes)
@@
 			)
 		)
-		(property "Value" "10M"
+		(property "Value" "10M 5%"
 			(at 211.67 61.79 0)
 			(show_name no)
@@
 			)
 		)
-		(property "Footprint" "Resistor_SMD:R_0603_1608Metric"
+		(property "Footprint" "Resistor_SMD:R_0402_1005Metric"
 			(at 214.122 60.96 90)
 			(hide yes)
@@
 			)
 		)
-		(property "LCSC" "C7250"
+		(property "LCSC" "C26086"
 			(at 215.9 60.96 0)
 			(hide yes)
@@
 			)
 		)
-		(property "MPN" "0603WAF1005T5E"
+		(property "MPN" "0402WGJ0106TCE"
 			(at 215.9 60.96 0)
 			(hide yes)
