File: Production/gauge.kicad_sch (KiCad schematic)
At the start: 65 parts, among them J102 Cell 1 NTC wires, J105 Cell 2 NTC wires, J106 Cell 3 NTC wires, J107 Cell 4 NTC wires, J108 PACK- (CELL_N), J109 CELL1 tap, J110 CELL2 tap, J111 CELL3 tap, J112 PACK+ (CELL_P_RAW), Q101 AGM404AP1, Q102 AGM404AP1, Q103 AO3400A, Q104 AO3400A, U101 BQ40Z50RSMR-R2, U102 BQ294700DSGR

Commit message: Production P0 is the first build: gauge training access and tuning hedges
Dev board skipped. J302 = second TC2030-NL (GAUGE: SDA, CHG_INH, NRST, GND,
SCL) replacing the SMBus pogo pads; J113/J114 PACK_P/GND load pads for the
learning cycle; R118 4.7k + TP113 WAKE pad. Hedges: R444-R447 back as 0R
0402 gate links, DNP 0402 snubbers. Probe pads (1.0 mm) VBUS/PPHV/PP5V/REGN/
SW1/SW2/GND per port. docs/production/p0-bringup-and-training.md. Netlist
check passes; ERC known warnings only. Board/.kicad_pro (user WIP) not included.

Co-Authored-By: Claude Opus 5.5 <noreply@anthropic.com>
Parts:
- removed TP110: SMBC, TestPoint:TestPoint_Pad_D1.5mm, symbol Connector:TestPoint
- removed TP111: SMBD, TestPoint:TestPoint_Pad_D1.5mm, symbol Connector:TestPoint
- removed TP112: GND, TestPoint:TestPoint_Pad_D1.5mm, symbol Connector:TestPoint
- added J113: LOAD PACK_P, Connector_Wire:SolderWire-0.5sqmm_1x01_D0.9mm_OD2.1mm, symbol Connector:TestPoint
- added J114: LOAD GND, Connector_Wire:SolderWire-0.5sqmm_1x01_D0.9mm_OD2.1mm, symbol Connector:TestPoint
- added R118: 4.7k, Resistor_SMD:R_0402_1005Metric, symbol Device:R
- added TP113: WAKE, TestPoint:TestPoint_Pad_D1.0mm, symbol Connector:TestPoint
- TP106, TP109: footprint TestPoint:TestPoint_Pad_D1.5mm -> TestPoint:TestPoint_Pad_D1.0mm
Connections:
- net CELL_P: now also R118.1
- net GND: now also J114.1
- net PACK_P: now also J113.1
- new net WAKE: R118.2, TP113.1
Other:
- note added: "Training: J113/J114 = learning-cycle load wires (20 AWG). WAKE: bridge TP113 to TP106 (PACK_P)."

Commit message: Production schematic P0: layout clean-up pass
New tools/layout_production.py (after make and tidy): block moves via
DevBoard/tools/move_region.py, then place_fields.py and check_overlaps.py.
Gauge: pack/NTC pads compacted, current sense and test/training pads moved up;
MCU: blocks regrouped, notes moved, J302 at 5.08 mm pin pitch; 3V3 Rail:
shared bulk and notes beside the rail; stale headings and index text fixed.
0 overlaps on all sheets; netlist check passes; ERC known warnings only.

Co-Authored-By: Claude Opus 5.5 <noreply@anthropic.com>
Parts:
- J108: value PACK- (CELL_N) -> PACK-; Notes (none) -> CELL_N
- J112: value PACK+ (CELL_P_RAW) -> PACK+; Notes (none) -> CELL_P_RAW
Other:
- note added: "GAUGE SMBus (0x0B): access via J302 on the MCU sheet"
- note added: "TEST + TRAINING PADS"
- note removed: "FACTORY TEST PADS"
- note removed: "GAUGE SMBus (0x0B) + POGO PADS"
- moved on the sheet: C106, J102, J105, J106, J107, R107, R108, RS101, TP106, TP109
