File: Production/mcu.kicad_sch (KiCad schematic)
At the start: 16 parts, among them J301 TC2030-NL, U301 CC2340R5MODA

Commit message: Production schematic P0: drawing tidy
tools/tidy_production.py (runs after make_production.py): pogo pads in their
own row, TC2030 under its SWD heading, link-merge leftovers removed, empty
headings deleted, sheet notes, root index and revision log rewritten for
production, sheets renamed 3V3 Rail and MCU. Netlist unchanged (check_netlist
passes); ERC: no errors.

Co-Authored-By: Claude Opus 5.5 <noreply@anthropic.com>
Other:
- note added: "3V3_SLEEP PULL-UP"
- note added: "FACTORY TEST PAD"
- note added: "NOTES 1. U301 antenna end at a board edge, ground 10-20 mm each side; keep-out in the footprint (fig. 9-2). 2. C301-C303 at the VDDS pads. R302 + C304 = power-on reset (SWRS349A fig. 9-1 R1/C92); no reset button. 3. C313 = CA1. R321/C314/C315 = Z61/Z60/Z62 pi match (TI: 0R, DNP, 1 pF); retune on the board. 4. No 32 kHz crystal: LFOSC calibrated against the 48 MHz crystal. DIO3/DIO4 are GPIOs. 5. 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"
- note added: "SWD (Tag-Connect TC2030-NL)"
- note removed: "BRING-UP AIDS"
- note removed: "DEBUG HEADERS"
- note removed: "NOTES 1. U301 antenna end at a board edge, ground 10-20 mm each side; keep-out in the footprint (fig. 9-2). 2. C301-C303 at the VDDS pads. R302 + C304 = power-on reset (SWRS349A fig. 9-1 R1/C92). 3. C313 = CA1. R321/C314/C315 = Z61/Z60/Z62 pi match (TI: 0R, DNP, 1 pF); retune on the board. 4. No 32 kHz crystal: LFOSC calibrated against the 48 MHz crystal. DIO3/DIO4 are GPIOs. 5. Pins: DIO6 SCL, D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"
- note removed: "STATUS LED"
- note removed: "TEST POINTS"

Commit message: Production schematic P0: passive downsizing (-432 mm2 courtyard, -16 %)
Extended parts and 0201 allowed on production (0201 only where both nets stay
<= 5.5 V). Charger inductor 10x10 -> Coilank APS0730M2R2F; 0603 R -> 0402;
low-voltage R/C -> 0201; RAC 0805, RBAT 1206, gauge shunt 1206; R101-R104
0402; BAT54 SOD-882; REGN/filter/SS caps 0402; NTC 0402. Bulk polymers and
TPS25751/TPS62933 caps kept (leakage, derating). New APS0730 footprint is
written by make_production.py. Netlist check passes; ERC clean.

Co-Authored-By: Claude Opus 5.5 <noreply@anthropic.com>
Parts:
- C302, C303, C304: value 0.1u 50V -> 0.1u 16V; footprint Capacitor_SMD:C_0402_1005Metric -> Capacitor_SMD:C_0201_0603Metric; LCSC C307331 -> C307380; MPN CL05B104KB54PNC -> CL03A104KO3NNNC
- R302: footprint Resistor_SMD:R_0402_1005Metric -> Resistor_SMD:R_0201_0603Metric; LCSC C25741 -> C270364; MPN 0402WGF1003TCE -> 0201WMF1003TEE
- R304, R305: footprint Resistor_SMD:R_0402_1005Metric -> Resistor_SMD:R_0201_0603Metric; LCSC C25890 -> C270350; MPN 0402WGF3301TCE -> 0201WMF3301TEE
- R313: footprint Resistor_SMD:R_0603_1608Metric -> Resistor_SMD:R_0201_0603Metric; LCSC C22961 -> C473458; MPN 0603WAF2203T5E -> 0201WMF2203TEE
- R314: footprint Resistor_SMD:R_0402_1005Metric -> Resistor_SMD:R_0201_0603Metric; LCSC C25792 -> C270345; MPN 0402WGF4702TCE -> 0201WMF4702TEE
Changed lines of the file:
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@@
 			)
 		)
-		(property "Footprint" "Resistor_SMD:R_0402_1005Metric"
+		(property "Footprint" "Resistor_SMD:R_0201_0603Metric"
 			(at 264.16 190.5 0)
 			(hide yes)
@@
 			)
 		)
-		(property "LCSC" "C25792"
+		(property "LCSC" "C270345"
 			(at 264.16 190.5 0)
 			(hide yes)
@@
 			)
 		)
-		(property "MPN" "0402WGF4702TCE"
+		(property "MPN" "0201WMF4702TEE"
 			(at 264.16 190.5 0)
 			(hide yes)
@@
 			)
 		)
-		(property "Footprint" "Resistor_SMD:R_0603_1608Metric"
+		(property "Footprint" "Resistor_SMD:R_0201_0603Metric"
 			(at 81.28 44.45 0)
 			(hide yes)
@@
 			)
 		)
-		(property "LCSC" "C22961"
+		(property "LCSC" "C473458"
 			(at 81.28 44.45 0)
 			(hide yes)
@@
 			)
 		)
-		(property "MPN" "0603WAF2203T5E"
+		(property "MPN" "0201WMF2203TEE"
 			(at 81.28 44.45 0)
 			(hide yes)
@@
 			)
 		)
-		(property "Value" "0.1u 50V"
+		(property "Value" "0.1u 16V"
 			(at 151.13 99.67 0)
 			(show_name no)
@@
 			)
 		)
-		(property "Footprint" "Capacitor_SMD:C_0402_1005Metric"
+		(property "Footprint" "Capacitor_SMD:C_0201_0603Metric"
 			(at 150.825 101.6 0)
 			(hide yes)
@@
 			)
 		)
-		(property "LCSC" "C307331"
+		(property "LCSC" "C307380"
 			(at 149.86 105.41 0)
 			(hide yes)
@@
 			)
 		)
-		(property "MPN" "CL05B104KB54PNC"
+		(property "MPN" "CL03A104KO3NNNC"
 			(at 149.86 105.41 0)
 			(hide yes)
@@
 			)
 		)
-		(property "Footprint" "Resistor_SMD:R_0402_1005Metric"
+		(property "Footprint" "Resistor_SMD:R_0201_0603Metric"
 			(at 152.4 120.65 0)
 			(hide yes)
@@
 			)
 		)
-		(property "LCSC" "C25741"
+		(property "LCSC" "C270364"
 			(at 152.4 120.65 0)
 			(hide yes)
@@
 			)
 		)
-		(property "MPN" "0402WGF1003TCE"
+		(property "MPN" "0201WMF1003TEE"
 			(at 152.4 120.65 0)
 			(hide yes)
@@
 			)
 		)
-		(property "Footprint" "Resistor_SMD:R_0402_1005Metric"
+		(property "Footprint" "Resistor_SMD:R_0201_0603Metric"
 			(at 231.902 190.5 90)
 			(hide yes)
@@
 			)
 		)
-		(property "LCSC" "C25890"
+		(property "LCSC" "C270350"
 			(at 233.68 190.5 0)
 			(hide yes)
@@
 			)
 		)
-		(property "MPN" "0402WGF3301TCE"
+		(property "MPN" "0201WMF3301TEE"
 			(at 233.68 190.5 0)
 			(hide yes)
@@
 			)
 		)
-		(property "Footprint" "Resistor_SMD:R_0402_1005Metric"
+		(property "Footprint" "Resistor_SMD:R_0201_0603Metric"
 			(at 247.142 190.5 90)
 			(hide yes)
@@
 			)
 		)
-		(property "LCSC" "C25890"
+		(property "LCSC" "C270350"
 			(at 248.92 190.5 0)
 			(hide yes)
@@
 			)
 		)
-		(property "MPN" "0402WGF3301TCE"
+		(property "MPN" "0201WMF3301TEE"
 			(at 248.92 190.5 0)
 			(hide yes)
@@
 			)
 		)
-		(property "Value" "0.1u 50V"
+		(property "Value" "0.1u 16V"
 			(at 145.9 120.64 90)
 			(show_name no)
@@
 			)
 		)
-		(property "Footprint" "Capacitor_SMD:C_0402_1005Metric"
+		(property "Footprint" "Capacitor_SMD:C_0201_0603Metric"
 			(at 149.555 120.65 0)
 			(hide yes)
@@
 			)
 		)
-		(property "LCSC" "C307331"
+		(property "LCSC" "C307380"
 			(at 148.59 124.46 0)
 			(hide yes)
@@
 			)
 		)
-		(property "MPN" "CL05B104KB54PNC"
+		(property "MPN" "CL03A104KO3NNNC"
 			(at 148.59 124.46 0)
 			(hide yes)
@@
 			)
 		)
-		(property "Value" "0.1u 50V"
+		(property "Value" "0.1u 16V"
 			(at 161.29 99.67 0)
 			(show_name no)
@@
 			)
 		)
-		(property "Footprint" "Capacitor_SMD:C_0402_1005Metric"
+		(property "Footprint" "Capacitor_SMD:C_0201_0603Metric"
 			(at 160.985 101.6 0)
 			(hide yes)
@@
 			)
 		)
-		(property "LCSC" "C307331"
+		(property "LCSC" "C307380"
 			(at 160.02 105.41 0)
 			(hide yes)
@@
 			)
 		)
-		(property "MPN" "CL05B104KB54PNC"
+		(property "MPN" "CL03A104KO3NNNC"
 			(at 160.02 105.41 0)
 			(hide yes)
