File: Production/Monolith.kicad_pcb (KiCad board)
At the start: 6 copper layers, 45.5 x 45.5 mm, 246 parts, among them J102 Cell 1 NTC wires, J105 Cell 2 NTC wires, J106 Cell 3 NTC wires, J107 Cell 4 NTC wires, J108 PACK- (CELL_N), J109 CELL1 tap, J110 CELL2 tap, J111 CELL3 tap, J112 PACK+ (CELL_P_RAW), J301 TC2030-NL, J401 TYPE-C 16PCB0.8 IP68, J501 TYPE-C 16PCB0.8 IP68, Q101 AGM404AP1, Q102 AGM404AP1, Q103 AO3400A, Q104 AO3400A, Q401 SiZ240DT, Q402 SiZ240DT, Q501 SiZ240DT, Q502 SiZ240DT, U101 BQ40Z50RSMR-R2, U102 BQ294700DSGR, U204 TPS62177DQCR, U301 CC2340R5MODA, U401 TPS25751DREFR, U402 M24512-DFMC6TG, U403 BQ25756RRVR, U404 TPS62933DRLR, U405 TPD2S300YFFR, U501 TPS25751DREFR, U502 M24512-DFMC6TG, U503 BQ25756RRVR, U504 TPS62933DRLR, U505 TPD2S300YFFR

Commit message: Production changes to still generate golden file and skip proto board
Parts:
- moved U405 135.5 mm to (110.4, 113.4)
- moved U401 113.8 mm to (110.5, 104.3), turned to -90 degrees
Routing:
- net /USB Port 1/VBUS: track 0.00 -> 8.89 mm
