File: Production/usb_port.kicad_sch (KiCad schematic)
At the start: 96 parts, among them J401 TYPE-C 16PCB1.6 IP68, Q401 SiZ240DT, Q402 SiZ240DT, U401 TPS25751DREFR, U402 M24512-DFMC6TG, U403 BQ25756RRVR, U404 TPS62933DRLR, U405 TPD6S300RUKR

Commit message: Production: USB bulk -> 2x CA55-D035M476T 47u polymer tantalum
Per port 4x 22u 1210 + 2x CCTC CA55-D035M476T (C421, C456; C457 dropped):
99.7 uF worst at 20 V, damping 20.0 dB, 2.8 mm max, $1.49 each instead of
three $3.20 T521Ds. The CA45 MnO2 version was rejected: fails short and can
ignite, and would run above its 50 % derating on a USB input
(low_profile_sims.py C2, CA45 and CA55 options added).

Co-Authored-By: Claude Opus 5.5 <noreply@anthropic.com>
Parts:
- removed C457: 33u 35V, Capacitor_Tantalum_SMD:CP_EIA-7343-31_Kemet-D, symbol Device:C_Polarized
- C421: value 33u 35V -> 47u 35V; LCSC C696815 -> C2761440; MPN KEMET T521D336M035ATE065 (polymer tantalum) -> CCTC CA55-D035M476T (polymer tantalum); Notes USB-side bulk with C456/C457 (three 33 uF polymer tantalum,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 -> USB-side bulk with C456 (two 47 uF 35 V polymer tantalum, 1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
- C456: value 33u 35V -> 47u 35V; LCSC C696815 -> C2761440; MPN KEMET T521D336M035ATE065 (polymer tantalum) -> CCTC CA55-D035M476T (polymer tantalum); Notes T521D on AC_SNS_N with C421, see C421 -> Second CA55 47u on AC_SNS_N, see C421
