File: hardware/Production/Monolith.kicad_pcb (KiCad board)
At the start: 6 copper layers, 43.2 x 74.4 mm, 289 parts, among them J102 Cell 1 NTC wires, J105 Cell 2 NTC wires, J106 Cell 3 NTC wires, J107 Cell 4 NTC wires, J108 PACK- power slot, J109 CELL1 slot, J110 CELL2 slot, J111 CELL3 slot, J112 PACK+ power slot, J113 LOAD PACK_P, J114 LOAD GND, J115 1N Kelvin slot, J116 4P Kelvin slot, J301 TC2030-NL, J302 TC2030-NL GAUGE, J401 TYPE-C 16PCB1.6 IP68, J501 TYPE-C 16PCB1.6 IP68, Q101 AGM404AP1, Q102 AGM404AP1, Q103 AO3400A, Q104 AO3400A, Q401 SiZ240DT, Q402 SiZ240DT, Q501 SiZ240DT, Q502 SiZ240DT, U101 BQ40Z50RSMR-R2, U102 BQ294700DSGR, U204 TPS62177DQCR, U301 CC2340R5MODA, U401 TPS25751DREFR, U402 M24512-DFMC6TG, U403 BQ25756RRVR, U404 TPS62933DRLR, U405 TPD6S300RUKR, U501 TPS25751DREFR, U502 M24512-DFMC6TG, U503 BQ25756RRVR, U504 TPS62933DRLR, U505 TPD6S300RUKR

Commit message: Placement In Progress
Parts:
- U301: moved to F.Cu
- moved U301 96.3 mm to (116.3, 122.2), turned to -90 degrees
- moved C427 52.5 mm to (105.0, 87.8)
- moved C424 52.5 mm to (101.7, 87.8)
- moved D405 47.8 mm to (113.2, 91.1), turned to 90 degrees
- moved D404 47.3 mm to (113.0, 99.6), turned to -90 degrees
- moved R412 47.2 mm to (119.1, 100.0), turned to -90 degrees
- moved R435 45.2 mm to (120.8, 95.3), turned to 90 degrees
- moved R417 43.3 mm to (121.5, 97.2), turned to 180 degrees
- moved L401 41.2 mm to (104.3, 94.4), turned to -90 degrees
- moved U402 41.0 mm to (103.1, 83.8), turned to 180 degrees
- moved C423 40.6 mm to (109.2, 86.7), turned to 90 degrees
- moved R428 34.9 mm to (117.3, 88.6), turned to -90 degrees
- moved C420 34.7 mm to (114.6, 87.4), turned to -90 degrees
- moved C431 33.7 mm to (110.0, 102.4)
- moved R429 33.5 mm to (118.4, 88.6), turned to -90 degrees
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