File: hardware/Production/Monolith.kicad_pcb (KiCad board)
At the start: 6 copper layers, 43.2 x 74.4 mm, 289 parts, among them J102 Cell 1 NTC wires, J105 Cell 2 NTC wires, J106 Cell 3 NTC wires, J107 Cell 4 NTC wires, J108 PACK- power wire, J109 CELL1 slot, J110 CELL2 slot, J111 CELL3 slot, J112 PACK+ power wire, J113 LOAD PACK_P, J114 LOAD GND, J115 1N Kelvin slot, J116 4P Kelvin slot, J301 TC2030-NL, J302 TC2030-NL GAUGE, J401 TYPE-C 16PCB1.6 IP68, J501 TYPE-C 16PCB1.6 IP68, Q101 AGM404AP1, Q102 AGM404AP1, Q103 AO3400A, Q104 AO3400A, Q401 SiZ240DT, Q402 SiZ240DT, Q501 SiZ240DT, Q502 SiZ240DT, U101 BQ40Z50RSMR-R2, U102 BQ294700DSGR, U204 TPS62177DQCR, U301 CC2340R5MODA, U401 TPS25751DREFR, U402 M24512-DFMC6TG, U403 BQ25756RRVR, U404 TPS62933DRLR, U405 TPD6S300RUKR, U501 TPS25751DREFR, U502 M24512-DFMC6TG, U503 BQ25756RRVR, U504 TPS62933DRLR, U505 TPD6S300RUKR

Commit message: Sense leads as wires; cup, cap and carrier fixes from the 2026-10-24 review
Sense wires (Logan): CELL1-3 become 28 AWG PTFE wires like the 1N / 4P
Kelvin leads. CELL1 / CELL3 solder to a short tongue of the top strip just
past the top frame; CELL2 solders to the middle of the bottom strip and runs
in a channel in the bottom frame. The five board pads keep their copper and
get a round 0.8 mm drill instead of the oval slot (J109-J111, J115, J116).

Review fixes in monolith_cup.py:
- cap: outer collar with crush ribs holds the mouth against the O-ring;
  O-ring and screws moved up so each screw has a 1.2 mm ligament; blind
  pilots (no path round the seal); skirt 2.6 mm (1.2 mm root), its top
  1.1 mm under the frame; four overtravel posts; pad printed 1.2 proud and
  relieved under the PACK pads
- carrier: board rails are four clip-on blocks keyed into the frames, so
  the front cells can be loaded; one merged wire notch per side (no loose
  chip); foam preload pockets; CELL2 channel
- peg posts run on to 0.3 mm under a 2.0 mm board-face wall; TPU sleeves
  hold the board on them
- fish-paper insulator rings on the four + ends
- top wall 1.85 mm; USB-C bores sized to the rev A4 ring with 0.15 mm
  squeeze and a lead-in
- new checks: one-piece parts, ligament, blind pilots, skirt gap, preload,
  wall deflection, key slots, channel

Board: R124 / R126 DNP (gauge note 16), so Q104 can't fire F102 while the
pack is wired up.

Co-Authored-By: Claude Opus 5.5 (1M context) <noreply@anthropic.com>
Claude-Session: https://claude.ai/code/session_01V2XuchjL8SPbkwDuzZLoSy
Parts:
- J109: value CELL1 slot -> CELL1 sense wire; footprint MonolithDev:Slot_Tab_3.4x0.6mm -> MonolithDev:SolderWire-28AWG_PTFE_1x01_D0.8mm_Pad4.2x1.4mm
- J110: value CELL2 slot -> CELL2 sense wire; footprint MonolithDev:Slot_Tab_3.4x0.6mm -> MonolithDev:SolderWire-28AWG_PTFE_1x01_D0.8mm_Pad4.2x1.4mm
- J111: value CELL3 slot -> CELL3 sense wire; footprint MonolithDev:Slot_Tab_3.4x0.6mm -> MonolithDev:SolderWire-28AWG_PTFE_1x01_D0.8mm_Pad4.2x1.4mm
- J115: value 1N Kelvin slot -> 1N Kelvin wire; footprint MonolithDev:Slot_Tab_1.6x0.6mm -> MonolithDev:SolderWire-28AWG_PTFE_1x01_D0.8mm_Pad2.4x1.4mm
- J116: value 4P Kelvin slot -> 4P Kelvin wire; footprint MonolithDev:Slot_Tab_1.6x0.6mm -> MonolithDev:SolderWire-28AWG_PTFE_1x01_D0.8mm_Pad2.4x1.4mm
Changed lines of the file:
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@@
 		)
 	)
-	(footprint "MonolithDev:Slot_Tab_1.6x0.6mm"
+	(footprint "MonolithDev:SolderWire-28AWG_PTFE_1x01_D0.8mm_Pad2.4x1.4mm"
 		(locked yes)
 		(layer "F.Cu")
 		(at 91.275 135.4755)
-		(descr "Plated slot 1.6 x 0.6 mm, 0.4 mm ring, for a nickel tail soldered on F.Cu (mechanical/monolith_shell.py sb_slots)")
-		(tags "slot nickel tab battery")
+		(descr "Plated hole 0.8 mm in a 2.4 x 1.4 mm pad, for a 28 AWG PTFE sense wire soldered on F.Cu (mechanical/monolith_shell.py sb_slots)")
+		(tags "connector wire 28AWG PTFE battery sense")
 		(property "Reference" "J115"
 			(at 0 -1.4 0)
@@
 			)
 		)
-		(property "Value" "1N Kelvin slot"
+		(property "Value" "1N Kelvin wire"
 			(at 0 1.4 0)
 			(layer "F.Fab")
@@
 			(at 0 0)
 			(size 2.4 1.4)
-			(drill oval 1.6 0.6)
+			(drill 0.8)
 			(layers "*.Cu" "*.Mask")
 			(remove_unused_layers no)
@@
 		)
 	)
-	(footprint "MonolithDev:Slot_Tab_3.4x0.6mm"
+	(footprint "MonolithDev:SolderWire-28AWG_PTFE_1x01_D0.8mm_Pad4.2x1.4mm"
 		(locked yes)
 		(layer "F.Cu")
 		(at 100 135.4505)
-		(descr "Plated slot 3.4 x 0.6 mm, 0.4 mm ring, for a nickel tail soldered on F.Cu (mechanical/monolith_shell.py sb_slots)")
-		(tags "slot nickel tab battery")
+		(descr "Plated hole 0.8 mm in a 4.2 x 1.4 mm pad, for a 28 AWG PTFE sense wire soldered on F.Cu (mechanical/monolith_shell.py sb_slots)")
+		(tags "connector wire 28AWG PTFE battery sense")
 		(property "Reference" "J110"
 			(at 0 -1.4 0)
@@
 			)
 		)
-		(property "Value" "CELL2 slot"
+		(property "Value" "CELL2 sense wire"
 			(at 0 1.4 0)
 			(layer "F.Fab")
@@
 			(at 0 0)
 			(size 4.2 1.4)
-			(drill oval 3.4 0.6)
+			(drill 0.8)
 			(layers "*.Cu" "*.Mask")
 			(remove_unused_layers no)
@@
 		)
 	)
-	(footprint "MonolithDev:Slot_Tab_3.4x0.6mm"
+	(footprint "MonolithDev:SolderWire-28AWG_PTFE_1x01_D0.8mm_Pad4.2x1.4mm"
 		(locked yes)
 		(layer "F.Cu")
 		(at 113.9 69.4755)
-		(descr "Plated slot 3.4 x 0.6 mm, 0.4 mm ring, for a nickel tail soldered on F.Cu (mechanical/monolith_shell.py sb_slots)")
-		(tags "slot nickel tab battery")
+		(descr "Plated hole 0.8 mm in a 4.2 x 1.4 mm pad, for a 28 AWG PTFE sense wire soldered on F.Cu (mechanical/monolith_shell.py sb_slots)")
+		(tags "connector wire 28AWG PTFE battery sense")
 		(property "Reference" "J111"
 			(at 0 -1.4 0)
@@
 			)
 		)
-		(property "Value" "CELL3 slot"
+		(property "Value" "CELL3 sense wire"
 			(at 0 1.4 0)
 			(layer "F.Fab")
@@
 			(at 0 0)
 			(size 4.2 1.4)
-			(drill oval 3.4 0.6)
+			(drill 0.8)
 			(layers "*.Cu" "*.Mask")
 			(remove_unused_layers no)
@@
 		)
 	)
-	(footprint "MonolithDev:Slot_Tab_3.4x0.6mm"
+	(footprint "MonolithDev:SolderWire-28AWG_PTFE_1x01_D0.8mm_Pad4.2x1.4mm"
 		(locked yes)
 		(layer "F.Cu")
 		(at 86.1 69.4755)
-		(descr "Plated slot 3.4 x 0.6 mm, 0.4 mm ring, for a nickel tail soldered on F.Cu (mechanical/monolith_shell.py sb_slots)")
-		(tags "slot nickel tab battery")
+		(descr "Plated hole 0.8 mm in a 4.2 x 1.4 mm pad, for a 28 AWG PTFE sense wire soldered on F.Cu (mechanical/monolith_shell.py sb_slots)")
+		(tags "connector wire 28AWG PTFE battery sense")
 		(property "Reference" "J109"
 			(at 0 -1.4 0)
@@
 			)
 		)
-		(property "Value" "CELL1 slot"
+		(property "Value" "CELL1 sense wire"
 			(at 0 1.4 0)
 			(layer "F.Fab")
@@
 			(at 0 0)
 			(size 4.2 1.4)
-			(drill oval 3.4 0.6)
+			(drill 0.8)
 			(layers "*.Cu" "*.Mask")
 			(remove_unused_layers no)
@@
 		)
 	)
-	(footprint "MonolithDev:Slot_Tab_1.6x0.6mm"
+	(footprint "MonolithDev:SolderWire-28AWG_PTFE_1x01_D0.8mm_Pad2.4x1.4mm"
 		(locked yes)
 		(layer "F.Cu")
 		(at 108.725 135.4755)
-		(descr "Plated slot 1.6 x 0.6 mm, 0.4 mm ring, for a nickel tail soldered on F.Cu (mechanical/monolith_shell.py sb_slots)")
-		(tags "slot nickel tab battery")
+		(descr "Plated hole 0.8 mm in a 2.4 x 1.4 mm pad, for a 28 AWG PTFE sense wire soldered on F.Cu (mechanical/monolith_shell.py sb_slots)")
+		(tags "connector wire 28AWG PTFE battery sense")
 		(property "Reference" "J116"
 			(at 0 -1.4 0)
@@
 			)
 		)
-		(property "Value" "4P Kelvin slot"
+		(property "Value" "4P Kelvin wire"
 			(at 0 1.4 0)
 			(layer "F.Fab")
@@
 			(at 0 0)
 			(size 2.4 1.4)
-			(drill oval 1.6 0.6)
+			(drill 0.8)
 			(layers "*.Cu" "*.Mask")
 			(remove_unused_layers no)
@@
 			)
 		)
-		(attr smd)
+		(attr smd dnp)
 		(duplicate_pad_numbers_are_jumpers no)
 		(fp_line
@@
 			)
 		)
-		(attr smd)
+		(attr smd dnp)
 		(duplicate_pad_numbers_are_jumpers no)
 		(fp_line
