File: hardware/Production/Monolith.kicad_pcb (KiCad board)
At the start: 6 copper layers, 43.2 x 74.4 mm, 289 parts, among them J102 Cell 1 NTC wires, J105 Cell 2 NTC wires, J106 Cell 3 NTC wires, J107 Cell 4 NTC wires, J108 PACK- power wire, J109 CELL1 sense wire, J110 CELL2 sense wire, J111 CELL3 sense wire, J112 PACK+ power wire, J113 LOAD PACK_P, J114 LOAD GND, J115 1N Kelvin wire, J116 4P Kelvin wire, J301 TC2030-NL, J302 TC2030-NL GAUGE, J401 TYPE-C 16PCB1.6 IP68, J501 TYPE-C 16PCB1.6 IP68, Q101 AGM404AP1, Q102 AGM404AP1, Q103 AO3400A, Q104 AO3400A, Q401 SiZ240DT, Q402 SiZ240DT, Q501 SiZ240DT, Q502 SiZ240DT, U101 BQ40Z50RSMR-R2, U102 BQ294700DSGR, U204 TPS62177DQCR, U301 CC2340R5MODA, U401 TPS25751DREFR, U402 M24512-DFMC6TG, U403 BQ25756RRVR, U404 TPS62933DRLR, U405 TPD6S300RUKR, U501 TPS25751DREFR, U502 M24512-DFMC6TG, U503 BQ25756RRVR, U504 TPS62933DRLR, U505 TPD6S300RUKR

Commit message: Layout in progress
Parts:
- removed R420, R520: 10R, Resistor_SMD:R_0402_1005Metric
- added C457: 1u 50V, Capacitor_SMD:C_0603_1608Metric, F.Cu at (118.6, 86.1)
- added C458: 22u 25V, Capacitor_SMD:C_0805_2012Metric, F.Cu at (118.6, 82.9)
- added C557: 1u 50V, Capacitor_SMD:C_0603_1608Metric, F.Cu at (161.6, 58.5)
- added C558: 22u 25V, Capacitor_SMD:C_0805_2012Metric, F.Cu at (156.9, 63.2)
- added D410: LRB520S-40T1G, Diode_SMD:D_SOD-523, F.Cu at (114.1, 106.0)
- added D411: LRB520S-40T1G, Diode_SMD:D_SOD-523, F.Cu at (118.5, 80.2)
- added D510: LRB520S-40T1G, Diode_SMD:D_SOD-523, F.Cu at (161.4, 61.0)
- added D511: LRB520S-40T1G, Diode_SMD:D_SOD-523, F.Cu at (161.4, 63.4)
- added Q409: AO3400A, Package_TO_SOT_SMD:SOT-23, F.Cu at (112.2, 84.5)
- added Q509: AO3400A, Package_TO_SOT_SMD:SOT-23, F.Cu at (157.1, 59.5)
- added R452: 40.2k 1%, Resistor_SMD:R_0402_1005Metric, F.Cu at (116.2, 80.2)
- added R453: 5.6k 1%, Resistor_SMD:R_0402_1005Metric, F.Cu at (114.2, 80.2)
- added R454: 100k, Resistor_SMD:R_0201_0603Metric, F.Cu at (112.2, 87.3)
- added R455: 100k, Resistor_SMD:R_0201_0603Metric, F.Cu at (113.2, 81.6)
- added R552: 40.2k 1%, Resistor_SMD:R_0402_1005Metric, F.Cu at (163.5, 53.6)
- added R553: 5.6k 1%, Resistor_SMD:R_0402_1005Metric, F.Cu at (163.5, 55.6)
- added R554: 100k, Resistor_SMD:R_0201_0603Metric, F.Cu at (164.4, 60.6)
- added R555: 100k, Resistor_SMD:R_0201_0603Metric, F.Cu at (164.4, 62.4)
- added U406: TPS7A4101DGNR, Package_SO:HVSSOP-8-1EP_3x3mm_P0.65mm_EP1.57x1.89mm, F.Cu at (115.7, 84.1)
- added U506: TPS7A4101DGNR, Package_SO:HVSSOP-8-1EP_3x3mm_P0.65mm_EP1.57x1.89mm, F.Cu at (158.3, 55.0)
- C411, C511: value 4.7u 10V -> 4.7u 25V; footprint Capacitor_SMD:C_0402_1005Metric -> Capacitor_SMD:C_0805_2012Metric
- L401, L501: value 2.2u -> 3.3u
- Q101, Q102: value AGM404AP1 -> BSC007N04LS6; footprint MonolithDev:AGM_PDFN-8_3.3x3.3mm_P0.65mm -> MonolithDev:Infineon_PG-TDSON-8_6.15x5.15mm_D5-8
- R412, R512: value 40.2k 1% -> 49.9k 1%
- moved R424 66.9 mm to (176.8, 94.0), turned to 90 degrees
- moved C409 66.0 mm to (106.0, 109.2), turned to 180 degrees
- moved R416 49.7 mm to (112.4, 115.0), turned to -90 degrees
- moved R409 49.1 mm to (106.6, 110.6), turned to 180 degrees
- moved R410 48.6 mm to (106.6, 111.8)
- moved R411 48.1 mm to (106.6, 112.9), turned to 180 degrees
- moved R427 44.5 mm to (118.2, 105.0), turned to -90 degrees
- moved R415 42.9 mm to (110.9, 116.0)
- moved TH401 40.5 mm to (111.8, 97.3)
- moved C421 32.8 mm to (133.7, 94.5)
- moved C410 31.8 mm to (109.9, 106.8), turned to 180 degrees
- moved C418 27.9 mm to (116.9, 108.8), turned to 90 degrees
- moved R413 26.9 mm to (113.4, 115.0)
- moved C411 25.8 mm to (115.9, 105.5), turned to 90 degrees
- moved R414 24.6 mm to (114.4, 115.0), turned to -90 degrees
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Connections:
- U401 pad 26: GND -> Net-(U401-GPIO4)
- U401 pad 27: GND -> Net-(U401-GPIO4)
- U401 pad 37: GND -> unconnected-(U401-GPIO6-Pad37)
- U501 pad 26: GND -> Net-(U501-GPIO4)
- U501 pad 27: GND -> Net-(U501-GPIO4)
- U501 pad 37: GND -> unconnected-(U501-GPIO6-Pad37)
Routing:
- net /USB Port 1/HG1: track 0.00 -> 1.52 mm
