File: hardware/Production/Monolith.kicad_pcb (KiCad board)
At the start: 6 copper layers, 43.2 x 74.4 mm, 287 parts, among them J105 Cell 2 NTC wires, J106 Cell 3 NTC wires, J108 PACK- power wire, J109 CELL1 sense wire, J110 CELL2 sense wire, J111 CELL3 sense wire, J112 PACK+ power wire, J113 LOAD PACK_P, J114 LOAD GND, J115 1N Kelvin wire, J116 4P Kelvin wire, J301 TC2030-NL, J302 TC2030-NL GAUGE, J401 TYPE-C 16PCB1.6 IP68, J501 TYPE-C 16PCB1.6 IP68, Q101 BSC007N04LS6, Q102 BSC007N04LS6, Q103 AO3400A, Q104 AO3400A, Q401 SiZ240DT, Q402 SiZ240DT, Q409 AO3400A, Q501 SiZ240DT, Q502 SiZ240DT, Q509 AO3400A, U101 BQ40Z50RSMR-R2, U102 BQ294700DSGR, U204 TPS62177DQCR, U301 CC2340R5MODA, U401 TPS25751DREFR, U402 M24512-DFMC6TG, U403 BQ25756RRVR, U404 TPS62933DRLR, U405 TPD6S300RUKR, U406 TPS7A4101DGNR, U501 TPS25751DREFR, U502 M24512-DFMC6TG, U503 BQ25756RRVR, U504 TPS62933DRLR, U505 TPD6S300RUKR, U506 TPS7A4101DGNR

Commit message: Backing Up before claude edit
Parts:
- moved R524 13.6 mm to (91.6, 80.7), turned to 0 degrees
- moved R555 0.29 mm to (93.7, 81.6)
Routing:
- net GND: track 0.00 -> 15.3 mm, vias 0 -> 138
- net /Cells and Gauge/CELL_1N: track 0.00 -> 13.9 mm, vias 0 -> 3
- net /USB Port 1/PP5V: track 0.00 -> 10.2 mm, vias 0 -> 3
- net /USB Port 2/PP5V: track 0.00 -> 9.92 mm, vias 0 -> 3
- net Net-(U101-VC1): track 0.00 -> 6.08 mm
- net /USB Port 2/SW_5V: track 0.00 -> 5.19 mm
- net /USB Port 1/SW_5V: track 0.00 -> 5.18 mm
- net /Cells and Gauge/BTP_INT: track 0.00 -> 4.91 mm, vias 0 -> 2
- net Net-(U101-VC2): track 0.00 -> 4.69 mm
- net /USB Port 1/PD_DRAIN: track 0.00 -> 4.48 mm
- net /USB Port 2/PD_DRAIN: track 0.00 -> 4.48 mm
- net Net-(U101-VC3): track 0.00 -> 4.41 mm
- net Net-(U101-VC4): track 0.00 -> 4.38 mm
- net /USB Port 2/PPHV: track 0.00 -> 4.06 mm, vias 0 -> 1
- net PACK_P: track 0.00 -> 4.04 mm
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- added copper zone on B.Cu, net /Cells and Gauge/FET_MID
- added copper zone on F.Cu, net /Cells and Gauge/FET_MID
- added copper zone on B.Cu, net /USB Port 1/AC_SNS_N
- added copper zone on F.Cu, net /USB Port 1/AC_SNS_N
- added copper zone on B.Cu, net /USB Port 1/BAT_SNS_P
- added copper zone on F.Cu, net /USB Port 1/BAT_SNS_P
- added copper zone on B.Cu, net /USB Port 1/PD_DRAIN
- added copper zone on F.Cu, net /USB Port 1/PPHV
- added copper zone on B.Cu, net /USB Port 1/SW1
- added copper zone on F.Cu, net /USB Port 1/SW1
- added copper zone on B.Cu, net /USB Port 1/SW2
- added copper zone on F.Cu, net /USB Port 1/SW2
- added copper zone on B.Cu, net /USB Port 1/VBUS
- added copper zone on F.Cu, net /USB Port 1/VBUS
- added copper zone on B.Cu, net /USB Port 2/AC_SNS_N
- added copper zone on F.Cu, net /USB Port 2/AC_SNS_N
- added copper zone on B.Cu, net /USB Port 2/BAT_SNS_P
- added copper zone on F.Cu, net /USB Port 2/BAT_SNS_P
- added copper zone on F.Cu, net /USB Port 2/PPHV
- added copper zone on B.Cu, net /USB Port 2/SW1
- added copper zone on F.Cu, net /USB Port 2/SW1
- added copper zone on B.Cu, net /USB Port 2/SW2
- added copper zone on F.Cu, net /USB Port 2/SW2
- added copper zone on B.Cu, net /USB Port 2/VBUS
- added copper zone on F.Cu, net /USB Port 2/VBUS
- added copper zone on B.Cu, net GND
- added copper zone on F.Cu, net GND
- added copper zone on In1.Cu, net GND

Commit message: more routing done
Parts:
- moved R517 0.38 mm to (87.8, 115.1)
- moved R535 0.38 mm to (87.7, 114.3)
- moved R305 0.36 mm to (109.9, 120.1)
- moved R513 0.13 mm to (90.4, 114.8)
- moved R514 0.13 mm to (91.4, 114.8)
- moved R516 0.13 mm to (89.4, 114.8)
Routing:
- net CELL_N: track 0.00 -> 53.3 mm, vias 0 -> 4
- net 3V3_SLEEP: track 0.00 -> 36.2 mm, vias 0 -> 2
- net /USB Port 2/DRV_SUP: track 0.00 -> 34.6 mm, vias 0 -> 4
- net CHG_INH: track 0.00 -> 31.4 mm, vias 0 -> 3
- net GND: track 15.3 -> 46.4 mm, vias 138 -> 186
- net /Cells and Gauge/CELL_1N: track 13.9 -> 44.9 mm, vias 3 -> 8
- net /USB Port 1/PPHV: track 0.20 -> 26.9 mm, vias 0 -> 2
- net /USB Port 2/REGN: track 0.00 -> 25.3 mm, vias 0 -> 3
- net /USB Port 1/AC_SNS_N: track 2.57 -> 27.0 mm, vias 24 -> 25
- net /USB Port 1/TS: track 0.00 -> 23.1 mm, vias 0 -> 3
- net /USB Port 2/TS: track 0.00 -> 22.2 mm, vias 0 -> 2
- net /MCU/NRST: track 0.00 -> 16.3 mm, vias 0 -> 2
- net PACK_P: track 4.04 -> 19.6 mm, vias 0 -> 24
- net /Cells and Gauge/CELL1: track 0.00 -> 14.1 mm, vias 0 -> 3
- net /USB Port 1/SW2: track 0.00 -> 13.0 mm, vias 32 -> 33
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- added copper zone on B.Cu, net /USB Port 2/PD_DRAIN
- added copper zone on In4.Cu, net GND
Other:
- board text added: "GAP FILLER"
- board text added: "GEL 30 2.3 g"

Commit message: Further routing work
Routing:
- net /Cells and Gauge/CELL3: track 0.00 -> 91.4 mm, vias 0 -> 3
- net /Cells and Gauge/CELL1: track 14.1 -> 82.2 mm
- net /P1_LDO_3V3: track 0.00 -> 30.2 mm, vias 0 -> 5
- net /USB Port 1/DRV_SUP: track 8.19 -> 38.3 mm, vias 3 -> 5
- net GND: track 46.4 -> 74.7 mm, vias 186 -> 202
- net 3V3: track 12.3 -> 37.6 mm, vias 16 -> 18
- net EN_5V2: track 2.65 -> 27.8 mm, vias 0 -> 4
- net /Cells and Gauge/CELL_4P: track 1.28 -> 24.7 mm, vias 0 -> 4
- net EN_5V1: track 0.00 -> 20.4 mm, vias 0 -> 3
- net /USB Port 1/SBU_FLT: track 0.00 -> 19.2 mm, vias 0 -> 3
- net /Cells and Gauge/CHG_G: track 1.45 -> 16.0 mm, vias 1 -> 2
- net /Cells and Gauge/CELL2: track 0.00 -> 12.6 mm, vias 0 -> 2
- net /USB Port 2/C_CC2: track 0.00 -> 11.3 mm
- net /USB Port 1/C_CC1: track 0.00 -> 11.2 mm, vias 0 -> 2
- net /USB Port 2/REGN: track 25.3 -> 35.2 mm, vias 3 -> 4
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- added copper zone on In3.Cu, net /USB Port 1/AC_SNS_N
- added copper zone on F.Cu, net PACK_P
- added copper zone on In2.Cu, net PACK_P

Commit message: Board Layout Done Going to review
Parts:
- removed J105: Cell 2 NTC wires, Connector_Wire:SolderWire-0.15sqmm_1x02_P4mm_D0.5mm_OD1.5mm
- removed J106: Cell 3 NTC wires, Connector_Wire:SolderWire-0.15sqmm_1x02_P4mm_D0.5mm_OD1.5mm
- added J1: Conn_01x01, MonolithDev:SolderWire-28AWG_PTFE_1x01_D0.8mm_Pad1.5x1.4mm, F.Cu at (114.0, 127.8)
- added J2: Conn_01x01, MonolithDev:SolderWire-28AWG_PTFE_1x01_D0.8mm_Pad1.5x1.4mm, F.Cu at (112.3, 127.8)
- added J3: Conn_01x01, MonolithDev:SolderWire-28AWG_PTFE_1x01_D0.8mm_Pad1.5x1.4mm, F.Cu at (103.6, 136.1)
- added J4: Conn_01x01, MonolithDev:SolderWire-28AWG_PTFE_1x01_D0.8mm_Pad1.5x1.4mm, F.Cu at (105.4, 136.1)
Routing:
- net IRQ_N: track 1.80 -> 83.3 mm, vias 0 -> 8
- net SCL: track 10.6 -> 90.7 mm, vias 2 -> 7
- net /Cells and Gauge/CELL_1N: track 50.8 -> 122.8 mm, vias 8 -> 13
- net SDA: track 19.3 -> 88.7 mm, vias 3 -> 7
- net GND: track 74.7 -> 123.2 mm, vias 202 -> 211
- net /USB Port 2/CHG_INT: track 1.21 -> 46.4 mm, vias 0 -> 5
- net 3V3: track 37.6 -> 82.1 mm, vias 18 -> 20
- net /USB Port 2/I2CC_SDA: track 1.68 -> 44.4 mm, vias 0 -> 4
- net /USB Port 2/I2CC_SCL: track 1.36 -> 42.9 mm, vias 0 -> 4
- net PACK_P: track 23.5 -> 62.2 mm, vias 35 -> 59
- net /USB Port 2/PPHV: track 3.54 -> 40.3 mm, vias 2 -> 5
- net /USB Port 1/I2CC_SDA: track 6.03 -> 41.3 mm, vias 2 -> 4
- net /USB Port 1/CHG_INT: track 1.21 -> 35.3 mm, vias 0 -> 2
- net /USB Port 1/I2CC_SCL: track 7.60 -> 41.3 mm, vias 2 -> 3
- net /USB Port 2/AC_SNS_N: track 5.62 -> 38.4 mm, vias 25 -> 27
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- added copper zone on B.Cu, net /Cells and Gauge/CELL_P
- added copper zone on F.Cu, net /Cells and Gauge/CELL_P
- added copper zone on F.Cu, net /USB Port 1/PP5V
- added copper zone on In3.Cu, net /USB Port 2/AC_SNS_N
- added copper zone on B.Cu, net /USB Port 2/PP5V
- added copper zone on In3.Cu, net 3V3
- added copper zone on B.Cu, net PACK_P
Other:
- board text added: "KO_NOTE B.Cu (faces the cells, hand-soldered): parts <= 2.3 mm tall; up to ~5 mm only in the centre strip x 96-104 or beyond 18mm from centre. No heat sources on B.Cu. Gap filler zones: solid copper + thermal vias to the power stages. F.Cu: parts <= 3.2 mm (cup wall 0.5 mm above)."
- board text removed: "KO_NOTE B.Cu (faces the cells, hand-soldered): parts <= 2.3 mm tall; up to ~5 mm only in the centre strip x 96-104 or beyond 18 mm from centre. No heat sources on B.Cu. Gap filler zones: solid copper + thermal vias to the power stages. F.Cu: parts <= 3.2 mm (cup wall 0.5 mm above)."

Commit message: More correction from AI review
Connections:
- U401 pad 26: Net-(U401-GPIO4) -> GND
- U401 pad 27: Net-(U401-GPIO4) -> GND
- U401 pad 37: unconnected-(U401-GPIO6-Pad37) -> /USB Port 1/DRV9_OFF
- U405 pad 7: GND -> /USB Port 1/C_CC1
- U405 pad 8: /USB Port 1/C_CC1 -> GND
- U501 pad 26: Net-(U501-GPIO4) -> GND
- U501 pad 27: Net-(U501-GPIO4) -> GND
- U501 pad 37: unconnected-(U501-GPIO6-Pad37) -> /USB Port 2/DRV9_OFF
- U505 pad 7: GND -> /USB Port 2/C_CC1
- U505 pad 8: /USB Port 2/C_CC1 -> GND
Routing:
- net /USB Port 2/DRV9_OFF: track 1.76 -> 19.7 mm, vias 0 -> 3
- net /USB Port 1/DRV9_OFF: track 1.72 -> 15.6 mm, vias 0 -> 2
- net GND: track 123.2 -> 126.1 mm, vias 211 -> 213
- net /Cells and Gauge/CELL1: track 84.0 -> 84.6 mm
- net PACK_P: vias 59 -> 62
