File: hardware/Production/gauge.kicad_sch (KiCad schematic)
At the start: 68 parts, among them J102 Cell 1 NTC wires, J105 Cell 2 NTC wires, J106 Cell 3 NTC wires, J107 Cell 4 NTC wires, J108 PACK- power wire, J109 CELL1 slot, J110 CELL2 slot, J111 CELL3 slot, J112 PACK+ power wire, J113 LOAD PACK_P, J114 LOAD GND, J115 1N Kelvin slot, J116 4P Kelvin slot, Q101 AGM404AP1, Q102 AGM404AP1, Q103 AO3400A, Q104 AO3400A, U101 BQ40Z50RSMR-R2, U102 BQ294700DSGR

Commit message: Sense leads as wires; cup, cap and carrier fixes from the 2026-10-24 review
Sense wires (Logan): CELL1-3 become 28 AWG PTFE wires like the 1N / 4P
Kelvin leads. CELL1 / CELL3 solder to a short tongue of the top strip just
past the top frame; CELL2 solders to the middle of the bottom strip and runs
in a channel in the bottom frame. The five board pads keep their copper and
get a round 0.8 mm drill instead of the oval slot (J109-J111, J115, J116).

Review fixes in monolith_cup.py:
- cap: outer collar with crush ribs holds the mouth against the O-ring;
  O-ring and screws moved up so each screw has a 1.2 mm ligament; blind
  pilots (no path round the seal); skirt 2.6 mm (1.2 mm root), its top
  1.1 mm under the frame; four overtravel posts; pad printed 1.2 proud and
  relieved under the PACK pads
- carrier: board rails are four clip-on blocks keyed into the frames, so
  the front cells can be loaded; one merged wire notch per side (no loose
  chip); foam preload pockets; CELL2 channel
- peg posts run on to 0.3 mm under a 2.0 mm board-face wall; TPU sleeves
  hold the board on them
- fish-paper insulator rings on the four + ends
- top wall 1.85 mm; USB-C bores sized to the rev A4 ring with 0.15 mm
  squeeze and a lead-in
- new checks: one-piece parts, ligament, blind pilots, skirt gap, preload,
  wall deflection, key slots, channel

Board: R124 / R126 DNP (gauge note 16), so Q104 can't fire F102 while the
pack is wired up.

Co-Authored-By: Claude Opus 5.5 (1M context) <noreply@anthropic.com>
Claude-Session: https://claude.ai/code/session_01V2XuchjL8SPbkwDuzZLoSy
Parts:
- J109: value CELL1 slot -> CELL1 sense wire; footprint MonolithDev:Slot_Tab_3.4x0.6mm -> MonolithDev:SolderWire-28AWG_PTFE_1x01_D0.8mm_Pad4.2x1.4mm
- J110: value CELL2 slot -> CELL2 sense wire; footprint MonolithDev:Slot_Tab_3.4x0.6mm -> MonolithDev:SolderWire-28AWG_PTFE_1x01_D0.8mm_Pad4.2x1.4mm
- J111: value CELL3 slot -> CELL3 sense wire; footprint MonolithDev:Slot_Tab_3.4x0.6mm -> MonolithDev:SolderWire-28AWG_PTFE_1x01_D0.8mm_Pad4.2x1.4mm
- J115: value 1N Kelvin slot -> 1N Kelvin wire; footprint MonolithDev:Slot_Tab_1.6x0.6mm -> MonolithDev:SolderWire-28AWG_PTFE_1x01_D0.8mm_Pad2.4x1.4mm
- J116: value 4P Kelvin slot -> 4P Kelvin wire; footprint MonolithDev:Slot_Tab_1.6x0.6mm -> MonolithDev:SolderWire-28AWG_PTFE_1x01_D0.8mm_Pad2.4x1.4mm
- R124, R126: now not fitted
Other:
- note added: "J108 PACK- / J112 PACK+: 18 AWG power wires in 1.5 mm holes. J115 1N / J116 4P: Kelvin wires from the same pads. J109-J111: CELL1-3 28 AWG sense wires. USB unplugged, in order: PACK-, 1N, CELL1, CELL2, CELL3, 4P, PACK+ (note 15)."
- note added: "NOTES 1. CELL_N = cell 1 negative at the PACK- power wire J108 (RS101, Q104). CELL_1N = gauge VSS, star-connected only at the 1N Kelvin wire hole J115 (TI SLUA660 2.3). GND = system ground, on the far side of RS101. 2. Kelvin-route SRP/SRN from the RS101 pads; R107/R108/C106 at the IC. RS101 is a 1206 1 W 75 ppm alloy part (P0). 3. VC taps are separate thin traces from the sense-wire holes J109-J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"
- note removed: "J108 PACK- / J112 PACK+: 18 AWG power wires in 1.5 mm holes. J115 1N / J116 4P: Kelvin wires from the same pads. J109-J111: CELL1-3 tails. USB unplugged, in order: PACK-, 1N, CELL1, CELL2, CELL3, 4P, PACK+ (note 15)."
- note removed: "NOTES 1. CELL_N = cell 1 negative at the PACK- power wire J108 (RS101, Q104). CELL_1N = gauge VSS, star-connected only at the 1N Kelvin slot J115 (TI SLUA660 2.3). GND = system ground, on the far side of RS101. 2. Kelvin-route SRP/SRN from the RS101 pads; R107/R108/C106 at the IC. RS101 is a 1206 1 W 75 ppm alloy part (P0). 3. VC taps are separate thin traces from the slots J109-J111. VC4 and the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"
Changed lines of the file:
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@@
 		(rev "P0")
 		(company "Monolith 100 W battery bank - production")
-		(comment 1 "Welded 4S pack slots, BQ40Z50-R2 gauge/protector, protection FETs")
+		(comment 1 "Welded 4S pack wires, BQ40Z50-R2 gauge/protector, protection FETs")
 		(comment 2 "Spec + open items: Production/README.md")
 		(comment 3 "P0: dev board rev A8 stripped by Production/tools/make_production.py; not reviewed")
@@
 		)
 	)
-	(text "NOTES\n1. CELL_N = cell 1 negative at the PACK- power wire J108 (RS101, Q104). CELL_1N = gauge VSS, star-connected only\n   at the 1N Kelvin slot J115 (TI SLUA660 2.3). GND = system ground, on the far side of RS101.\n2. Kelvin-route SRP/SRN from the RS101 pads; R107/R108/C106 at the IC. RS101 is a 1206 1 W 75 ppm alloy part (P0).\n3. VC taps are separate thin traces from the slots J109-J111. VC4 and the U102 V4/VDD filters are on CELL_4P,\n    the 4P Kelvin slot J116 (before F102 and off the power wire): fuse and wire drop are not read as cell voltage.\n4. TS1-TS4: one wired 10k NTC per cell on J102, J105-J107, taped to the cell at mid-height; insulated sensors only\n    (cans 0-12.6 V above VSS, TS 2.1 V max). PTC, PTCEN, PRES, DISP tied to VSS per datasheet.\n5. VCC fed from FET common drain via R106 (TI R13). PACK sense via R113 10k (TI R15).\n6. BAT fed from CELL_4P (cell top, before F102) via D101 + R105 (TI fig. 9-12).\n7. Diamonds are PWR_FLAGs (ERC only, no part): each sits where its rail is sourced through a passive part.\n8. Q103 buffers BTP_INT onto the shared open-drain IRQ_N (CC2340 DIO11): IRQ_N is low while BTP_INT is high.\n   Keep BTP disabled, or set BTP_POL = 1 with BTP_EN = 1, or IRQ_N is held low (review 4 D-2).\n9. D103 clamps Q102 VGS at 15 V in a hard short. The dev board's C109/D102 inrush options are not on P0.\n10. No wake button: the gauge leaves SHUTDOWN when PACK_P comes up (USB plugged in: TPS25751 dead-battery sink +\n    BQ25756 charging with 3V3 down, USB sheet note 11). P0 fallback: bridge TP113 (WAKE, R118 4.7k from CELL_P) to TP106.\n11. Gauge access is the GAUGE Tag-Connect J302 on the MCU sheet (SMBus + CHG_INH + NRST): BQStudio / EV2400 for\n    training, golden image and calibration. J113/J114 = 20 AWG load wires (PACK_P/GND) for the learning-cycle discharge.\n12. TP106 PACK_P and TP109 GND are 1.0 mm probe pads.\n13. ESD caps (TI): C110+C111 in series across the FET pair (fig. 9-2 C1/C2), C107+C108 across PACK+/PACK- (sec. 9.2.2.1.5).\n14. Second level (TI fig. 9-11): U102 BQ294700 (4.35 V/cell, CD 0.1u = 1-2 s) or the gauge FUSE pin turns Q104 on;\n    F102's heater then blows its fuse, permanently opening the cell top. F102 is also the pack's only overcurrent fuse.\n15. Solder the pack with USB unplugged: PACK-, then 1N and the taps bottom-up, 4P, PACK+ last: a floating tap can read\n    > 4.35 V, U102 trips after 1-2 s and F102 blows. Gauge data flash: COV Delay 1 s, Min Blow Fuse Voltage 10500 mV."
+	(text "NOTES\n1. CELL_N = cell 1 negative at the PACK- power wire J108 (RS101, Q104). CELL_1N = gauge VSS, star-connected only\n   at the 1N Kelvin wire hole J115 (TI SLUA660 2.3). GND = system ground, on the far side of RS101.\n2. Kelvin-route SRP/SRN from the RS101 pads; R107/R108/C106 at the IC. RS101 is a 1206 1 W 75 ppm alloy part (P0).\n3. VC taps are separate thin traces from the sense-wire holes J109-J111. VC4 and the U102 V4/VDD filters are on CELL_4P,\n    the 4P Kelvin wire hole J116 (before F102 and off the power wire): fuse and wire drop are not read as cell voltage.\n4. TS1-TS4: one wired 10k NTC per cell on J102, J105-J107, taped to the cell at mid-height; insulated sensors only\n    (cans 0-12.6 V above VSS, TS 2.1 V max). PTC, PTCEN, PRES, DISP tied to VSS per datasheet.\n5. VCC fed from FET common drain via R106 (TI R13). PACK sense via R113 10k (TI R15).\n6. BAT fed from CELL_4P (cell top, before F102) via D101 + R105 (TI fig. 9-12).\n7. Diamonds are PWR_FLAGs (ERC only, no part): each sits where its rail is sourced through a passive part.\n8. Q103 buffers BTP_INT onto the shared open-drain IRQ_N (CC2340 DIO11): IRQ_N is low while BTP_INT is high.\n   Keep BTP disabled, or set BTP_POL = 1 with BTP_EN = 1, or IRQ_N is held low (review 4 D-2).\n9. D103 clamps Q102 VGS at 15 V in a hard short. The dev board's C109/D102 inrush options are not on P0.\n10. No wake button: the gauge leaves SHUTDOWN when PACK_P comes up (USB plugged in: TPS25751 dead-battery sink +\n    BQ25756 charging with 3V3 down, USB sheet note 11). P0 fallback: bridge TP113 (WAKE, R118 4.7k from CELL_P) to TP106.\n11. Gauge access is the GAUGE Tag-Connect J302 on the MCU sheet (SMBus + CHG_INH + NRST): BQStudio / EV2400 for\n    training, golden image and calibration. J113/J114 = 20 AWG load wires (PACK_P/GND) for the learning-cycle discharge.\n12. TP106 PACK_P and TP109 GND are 1.0 mm probe pads.\n13. ESD caps (TI): C110+C111 in series across the FET pair (fig. 9-2 C1/C2), C107+C108 across PACK+/PACK- (sec. 9.2.2.1.5).\n14. Second level (TI fig. 9-11): U102 BQ294700 (4.35 V/cell, CD 0.1u = 1-2 s) or the gauge FUSE pin turns Q104 on;\n    F102's heater then blows its fuse, permanently opening the cell top. F102 is also the pack's only overcurrent fuse.\n15. Solder the pack with USB unplugged: PACK-, then 1N and the taps bottom-up, 4P, PACK+ last: a floating tap can read\n    > 4.35 V, U102 trips after 1-2 s and F102 blows. Gauge data flash: COV Delay 1 s, Min Blow Fuse Voltage 10500 mV.\n16. R124 / R126 are DNP from JLC (2026-10-24): with them off, neither U102 nor the gauge FUSE pin can turn Q104 on while\n    the pack is wired up. Fit them by hand only after all seven pack voltages read right at the pads."
 		(exclude_from_sim no)
 		(at 196.596 248.412 0)
@@
 		)
 	)
-	(text "J108 PACK- / J112 PACK+: 18 AWG power wires in 1.5 mm holes. J115 1N / J116 4P: Kelvin wires from the same pads.\nJ109-J111: CELL1-3 tails. USB unplugged, in order: PACK-, 1N, CELL1, CELL2, CELL3, 4P, PACK+ (note 15)."
+	(text "J108 PACK- / J112 PACK+: 18 AWG power wires in 1.5 mm holes. J115 1N / J116 4P: Kelvin wires from the same pads.\nJ109-J111: CELL1-3 28 AWG sense wires. USB unplugged, in order: PACK-, 1N, CELL1, CELL2, CELL3, 4P, PACK+ (note 15)."
 		(exclude_from_sim no)
 		(at 22.86 40.64 0)
@@
 		(on_board yes)
 		(in_pos_files yes)
-		(dnp no)
+		(dnp yes)
 		(property "Reference" "R124"
 			(at 323.70 122.18 90)
@@
 		(on_board yes)
 		(in_pos_files yes)
-		(dnp no)
+		(dnp yes)
 		(property "Reference" "R126"
 			(at 357.29 122.06 0)
@@
 			)
 		)
-		(property "Value" "CELL1 slot"
+		(property "Value" "CELL1 sense wire"
 			(at 38.10 83.05 0)
 			(show_name no)
@@
 			)
 		)
-		(property "Footprint" "MonolithDev:Slot_Tab_3.4x0.6mm"
+		(property "Footprint" "MonolithDev:SolderWire-28AWG_PTFE_1x01_D0.8mm_Pad4.2x1.4mm"
 			(at 43.18 88.9 0)
 			(hide yes)
@@
 			)
 		)
-		(property "Value" "CELL2 slot"
+		(property "Value" "CELL2 sense wire"
 			(at 38.10 72.89 0)
 			(show_name no)
@@
 			)
 		)
-		(property "Footprint" "MonolithDev:Slot_Tab_3.4x0.6mm"
+		(property "Footprint" "MonolithDev:SolderWire-28AWG_PTFE_1x01_D0.8mm_Pad4.2x1.4mm"
 			(at 43.18 78.74 0)
 			(hide yes)
@@
 			)
 		)
-		(property "Value" "CELL3 slot"
+		(property "Value" "CELL3 sense wire"
 			(at 38.10 62.73 0)
 			(show_name no)
@@
 			)
 		)
-		(property "Footprint" "MonolithDev:Slot_Tab_3.4x0.6mm"
+		(property "Footprint" "MonolithDev:SolderWire-28AWG_PTFE_1x01_D0.8mm_Pad4.2x1.4mm"
 			(at 43.18 68.58 0)
 			(hide yes)
@@
 			)
 		)
-		(property "Value" "1N Kelvin slot"
+		(property "Value" "1N Kelvin wire"
 			(at 55.88 90.67 0)
 			(show_name no)
@@
 			)
 		)
-		(property "Footprint" "MonolithDev:Slot_Tab_1.6x0.6mm"
+		(property "Footprint" "MonolithDev:SolderWire-28AWG_PTFE_1x01_D0.8mm_Pad2.4x1.4mm"
 			(at 60.96 96.52 0)
 			(hide yes)
@@
 			)
 		)
-		(property "Value" "4P Kelvin slot"
+		(property "Value" "4P Kelvin wire"
 			(at 57.15 52.57 0)
 			(show_name no)
@@
 			)
 		)
-		(property "Footprint" "MonolithDev:Slot_Tab_1.6x0.6mm"
+		(property "Footprint" "MonolithDev:SolderWire-28AWG_PTFE_1x01_D0.8mm_Pad2.4x1.4mm"
 			(at 60.96 58.42 0)
 			(hide yes)

Commit message: Sense pads 1.5 x 1.4: clear the USB-C courtyards and match the library
DRC flagged J109 / J111 courtyards overlapping J501 / J401 (the 4.2 mm oval
pads kept from the old tab slots) and all five sense footprints as not
matching the library (the board copies still had the slot outline on F.Fab).
Nothing is routed to them yet, so every sense pad is now Ø0.8 in a 1.5 x 1.4
pad (SB_SWIRE_PAD_L), one library footprint, with the board copies written
to match it. J109 / J111 courtyards end 0.05 mm short of the USB-C ones.

Co-Authored-By: Claude Opus 5.5 (1M context) <noreply@anthropic.com>
Claude-Session: https://claude.ai/code/session_01V2XuchjL8SPbkwDuzZLoSy
Parts:
- J109, J110, J111: footprint MonolithDev:SolderWire-28AWG_PTFE_1x01_D0.8mm_Pad4.2x1.4mm -> MonolithDev:SolderWire-28AWG_PTFE_1x01_D0.8mm_Pad1.5x1.4mm
- J115, J116: footprint MonolithDev:SolderWire-28AWG_PTFE_1x01_D0.8mm_Pad2.4x1.4mm -> MonolithDev:SolderWire-28AWG_PTFE_1x01_D0.8mm_Pad1.5x1.4mm
Changed lines of the file:
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@@
 			)
 		)
-		(property "Footprint" "MonolithDev:SolderWire-28AWG_PTFE_1x01_D0.8mm_Pad4.2x1.4mm"
+		(property "Footprint" "MonolithDev:SolderWire-28AWG_PTFE_1x01_D0.8mm_Pad1.5x1.4mm"
 			(at 43.18 88.9 0)
 			(hide yes)
@@
 			)
 		)
-		(property "Footprint" "MonolithDev:SolderWire-28AWG_PTFE_1x01_D0.8mm_Pad4.2x1.4mm"
+		(property "Footprint" "MonolithDev:SolderWire-28AWG_PTFE_1x01_D0.8mm_Pad1.5x1.4mm"
 			(at 43.18 78.74 0)
 			(hide yes)
@@
 			)
 		)
-		(property "Footprint" "MonolithDev:SolderWire-28AWG_PTFE_1x01_D0.8mm_Pad4.2x1.4mm"
+		(property "Footprint" "MonolithDev:SolderWire-28AWG_PTFE_1x01_D0.8mm_Pad1.5x1.4mm"
 			(at 43.18 68.58 0)
 			(hide yes)
@@
 			)
 		)
-		(property "Footprint" "MonolithDev:SolderWire-28AWG_PTFE_1x01_D0.8mm_Pad2.4x1.4mm"
+		(property "Footprint" "MonolithDev:SolderWire-28AWG_PTFE_1x01_D0.8mm_Pad1.5x1.4mm"
 			(at 60.96 96.52 0)
 			(hide yes)
@@
 			)
 		)
-		(property "Footprint" "MonolithDev:SolderWire-28AWG_PTFE_1x01_D0.8mm_Pad2.4x1.4mm"
+		(property "Footprint" "MonolithDev:SolderWire-28AWG_PTFE_1x01_D0.8mm_Pad1.5x1.4mm"
 			(at 60.96 58.42 0)
 			(hide yes)

Commit message: P0 schematic: protection FETs, 9 V gate drive and inductor loss cuts
The three board-side loss cuts approved on 2026-10-23 were in the spec
but never drawn. Now in the production schematic (port 1 refs):

- Cut 1: Q101/Q102 AGM404AP1 -> Infineon BSC007N04LS6 (C534274) on a
  5 x 6 footprint, KiCad's PG-TDSON-8 with the drain leads numbered 5-8
- Cut 2: 9 V DRV_SUP per port. U406 TPS7A4101 (C111739) from PACK_P,
  ~9.6 V via R452/R453, ORed onto DRV_SUP by D411; D410 replaces R420
  (REGN -> DRV_SUP) so the standard drive and dead-pack charging stay.
  EN = REGN via R454, held low by Q409 unless TPS25751 GPIO6 (DRV9_OFF,
  freed from the GND rail) is low: off by default, GPsl on, GPsh off.
  C411 -> 4.7u 25V 0805.
- Cut 3: L401 Coilcraft XGL7030-332 on the APS0730 pads, R412 49.9k
  (~500 kHz)

make_production.py builds all of it (add_gate_drive, free_gpio6,
tdson_footprint, tps7a4101.py); the committed sheets were updated with
the same functions since KiCad isn't available here. A script net diff
shows only the intended changes, and a regenerated usb/gauge sheet
matches. check_netlist.py knows the new nets. ERC and Update PCB from
Schematic are still to run in KiCad.

Co-Authored-By: Claude Opus 5.5 <noreply@anthropic.com>
Claude-Session: https://claude.ai/code/session_01LzE9uyZaPiG6jLirJVJbfw
Parts:
- Q101, Q102: value AGM404AP1 -> BSC007N04LS6; footprint MonolithDev:AGM_PDFN-8_3.3x3.3mm_P0.65mm -> MonolithDev:Infineon_PG-TDSON-8_6.15x5.15mm_D5-8; LCSC C41349455 -> C534274; MPN AGM404AP1 (AGMSEMI) -> BSC007N04LS6ATMA1 (Infineon)
Changed lines of the file:
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@@
 			)
 		)
-		(property "Value" "AGM404AP1"
+		(property "Value" "BSC007N04LS6"
 			(at 175.26 40.13 0)
 			(show_name no)
@@
 			)
 		)
-		(property "Footprint" "MonolithDev:AGM_PDFN-8_3.3x3.3mm_P0.65mm"
+		(property "Footprint" "MonolithDev:Infineon_PG-TDSON-8_6.15x5.15mm_D5-8"
 			(at 175.26 45.72 0)
 			(hide yes)
@@
 			)
 		)
-		(property "Datasheet" "https://www.lcsc.com/datasheet/C41349455.pdf"
+		(property "Datasheet" "https://www.lcsc.com/datasheet/C534274.pdf"
 			(at 175.26 45.72 0)
 			(hide yes)
@@
 			)
 		)
-		(property "Description" "40 V 4.4 mOhm N-MOSFET, PDFN3.3x3.3"
+		(property "Description" "40 V 0.7 mOhm N-MOSFET, TDSON-8 FL 5x6"
 			(at 175.26 45.72 0)
 			(hide yes)
@@
 			)
 		)
-		(property "LCSC" "C41349455"
+		(property "LCSC" "C534274"
 			(at 175.26 45.72 0)
 			(hide yes)
@@
 			)
 		)
-		(property "MPN" "AGM404AP1 (AGMSEMI)"
+		(property "MPN" "BSC007N04LS6ATMA1 (Infineon)"
 			(at 175.26 45.72 0)
 			(hide yes)
@@
 			)
 		)
-		(property "Value" "AGM404AP1"
+		(property "Value" "BSC007N04LS6"
 			(at 228.60 40.13 0)
 			(show_name no)
@@
 			)
 		)
-		(property "Footprint" "MonolithDev:AGM_PDFN-8_3.3x3.3mm_P0.65mm"
+		(property "Footprint" "MonolithDev:Infineon_PG-TDSON-8_6.15x5.15mm_D5-8"
 			(at 228.6 45.72 0)
 			(hide yes)
@@
 			)
 		)
-		(property "Datasheet" "https://www.lcsc.com/datasheet/C41349455.pdf"
+		(property "Datasheet" "https://www.lcsc.com/datasheet/C534274.pdf"
 			(at 228.6 45.72 0)
 			(hide yes)
@@
 			)
 		)
-		(property "Description" "40 V 4.4 mOhm N-MOSFET, PDFN3.3x3.3"
+		(property "Description" "40 V 0.7 mOhm N-MOSFET, TDSON-8 FL 5x6"
 			(at 228.6 45.72 0)
 			(hide yes)
@@
 			)
 		)
-		(property "LCSC" "C41349455"
+		(property "LCSC" "C534274"
 			(at 228.6 45.72 0)
 			(hide yes)
@@
 			)
 		)
-		(property "MPN" "AGM404AP1 (AGMSEMI)"
+		(property "MPN" "BSC007N04LS6ATMA1 (Infineon)"
 			(at 228.6 45.72 0)
 			(hide yes)
