File: hardware/Production/gauge.kicad_sch (KiCad schematic)
At the start: 68 parts, among them J105 Cell 2 NTC wires, J106 Cell 3 NTC wires, J108 PACK- power wire, J109 CELL1 sense wire, J110 CELL2 sense wire, J111 CELL3 sense wire, J112 PACK+ power wire, J113 LOAD PACK_P, J114 LOAD GND, J115 1N Kelvin wire, J116 4P Kelvin wire, Q101 BSC007N04LS6, Q102 BSC007N04LS6, Q103 AO3400A, Q104 AO3400A, U101 BQ40Z50RSMR-R2, U102 BQ294700DSGR

Commit message: Footprint Layout Done
Changed lines of the file:
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@@
 	(text "PACK SLOTS + WIRES  (welded 4S BAK 65E, tails and wires soldered on F.Cu)"
 		(exclude_from_sim no)
-		(at 22.86 33.02 0)
+		(at 12.7 24.384 0)
 		(effects
 			(font
@@
 	(symbol
 		(lib_id "Device:Thermistor_NTC")
-		(at 85.09 88.90 90)
+		(at 85.09 88.9 90)
 		(unit 1)
 		(body_style 1)
@@
 		)
 		(property "Footprint" "Resistor_SMD:R_0402_1005Metric"
-			(at 85.09 88.90 0)
+			(at 85.09 88.9 0)
 			(hide yes)
 			(show_name no)
@@
 		)
 		(property "Datasheet" ""
-			(at 85.09 88.90 0)
+			(at 85.09 88.9 0)
 			(hide yes)
 			(show_name no)
@@
 		)
 		(property "Description" "Temperature dependent resistor, negative temperature coefficient"
-			(at 85.09 88.90 0)
+			(at 85.09 88.9 0)
 			(hide yes)
 			(show_name no)
@@
 		)
 		(property "Notes" "Front-cell NTC, SMD on B.Cu in the outer bottom corner of the gap-filler zone over C4 (BT104), outboard of the BQ25756 (under the gel; research_notes/Pack thermal BAK 65E/smd-ntc.md). Reads the board there, 0.6-3.8 K above the hottest point of the C4 (BT104) can in the model. Keep the inner planes under it; low side to CELL_1N by its own trace. Gauge internal 18k pull-up; enable TS4 in data flash. Murata NCP15XH103F03RB/RC: B25/50 = 3380 K, B25/85 = 3435 K"
-			(at 85.09 88.90 0)
+			(at 85.09 88.9 0)
 			(hide yes)
 			(show_name no)
@@
 		)
 		(property "LCSC" "C77131"
-			(at 85.09 88.90 0)
+			(at 85.09 88.9 0)
 			(hide yes)
 			(show_name no)
@@
 		)
 		(property "MPN" "NCP15XH103F03RC"
-			(at 85.09 88.90 0)
-			(hide yes)
-			(show_name no)
+			(at 85.09 88.9 0)
+			(hide yes)
+			(show_name no)
