File: hardware/Production/usb_port.kicad_sch (KiCad schematic)
At the start: 104 parts, among them J401 TYPE-C 16PCB1.6 IP68, Q401 SiZ240DT, Q402 SiZ240DT, Q409 AO3400A, U401 TPS25751DREFR, U402 M24512-DFMC6TG, U403 BQ25756RRVR, U404 TPS62933DRLR, U405 TPD6S300RUKR, U406 TPS7A4101DGNR

Commit message: Layout in progress
Parts:
- added unit 1 of Q401
- added unit 2 of Q402
- Q401: Notes USB side high side (HIDRV1). JinYu PGQ04N070 (cost-down 202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 -> USB side low side (LODRV1). JinYu PGQ04N070 (cost-down 2026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
- Q402: Notes battery side low side (LODRV2). JinYu PGQ04N070 (cost-down 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 -> battery side high side (HIDRV2). JinYu PGQ04N070 (cost-down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
Connections:
- net AC_SNS_N: now also Q401.2 (D1), Q401.3 (D1), Q401.4 (D1); no longer Q401.2 (D1), Q401.3 (D1), Q401.4 (D1)
- net DRV9_OFF: no longer U401.37 (GPIO6)
- net GND: now also Q402.5 (S2), Q402.6 (S2), Q402.7 (S2); no longer Q402.5 (S2), Q402.6 (S2), Q402.7 (S2), U401.26 (GPIO4), U401.27 (GPIO5)
- net HG1: now also Q401.1 (G1); no longer Q401.1 (G1)
- net LG2: now also Q402.8 (G2); no longer Q402.8 (G2)
- net SW1: now also Q401.9 (SW)
- net SW2: now also Q402.9 (SW)
- new net: U401.26 (GPIO4), U401.27 (GPIO5)
Other:
- note removed: "U406 TPS7A4101 from PACK_P sets ~9.6 V (R452/R453); D411 ORs it onto DRV_SUP (~9.3 V). D410 (was R420 10R) feeds REGN - VF while U406 is off: TI's standard drive, so a dead pack still charges. EN = REGN via R454, held low by Q409 unless TPS25751 GPIO6 (DRV9_OFF) is low: GPIO6 Hi-Z or high = off. Configure GPIO6 as an output, initial high; 'GPsl' on, 'GPsh' off. Firmware: on only while this conver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"

Commit message: Footprint Layout Done
Parts:
- removed C454, C455: 33p C0G, Capacitor_SMD:C_0402_1005Metric, symbol Device:C
- removed R450, R451: 3R3, Resistor_SMD:R_0402_1005Metric, symbol Device:R

Commit message: Board Layout Done Going to review
Connections:
- net C_CC1: now also U405.7 (RPD_G1); no longer U405.8 (RPD_G1)
- net DRV9_OFF: now also U401.37 (GPIO6)
- net GND: now also U401.26 (GPIO4), U401.27 (GPIO5), U405.8 (GND); no longer U405.7 (GND)
Changed lines of the file:
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@@
+	)
+	(junction
+		(at 149.86 111.76)
+		(diameter 0)
+		(color 0 0 0 0)
+	)
+	(junction
+		(at 149.86 116.84)
+		(diameter 0)
+		(color 0 0 0 0)
 	)
 	(junction
@@
 	(no_connect
 		(at 138.43 166.37)
+	)
+	(wire
+		(pts
+			(xy 149.86 111.76) (xy 149.86 116.84)
+		)
+		(stroke
+			(width 0)
+			(type default)
+		)
+	)
+	(wire
+		(pts
+			(xy 154.94 114.3) (xy 144.78 114.3)
+		)
+		(stroke
+			(width 0)
+			(type default)
+		)
 	)
 	(wire
@@
 		)
 	)
+	(label "DRV9_OFF"
+		(at 144.78 114.3 180)
+		(effects
+			(font
+				(size 1.27 1.27)
+			)
+			(justify right bottom)
+		)
+	)

Commit message: Board Approved, Production Files Ready.
 Pending 3rd Party human review
Parts:
- L402: footprint MonolithDev:L_Coilank_APS0530 -> MonolithDev:L_COILMX_MS0520; LCSC C49073587 -> C49248023; MPN APS0530M3R3H (Coilank) -> EHE05023R3MFB (ABC); Notes Cost-down 2026-10-14 (was SRP5030T-3R3M): 3.3 uH, 38 mOhm m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 -> 2026-10-30 (was APS0530M3R3H, 3.1 mm tall, hit the cup corn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
Changed lines of the file:
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@@
 			)
 		)
-		(property "Footprint" "MonolithDev:L_Coilank_APS0530"
+		(property "Footprint" "MonolithDev:L_COILMX_MS0520"
 			(at 128.27 203.2 0)
 			(hide yes)
@@
 			)
 		)
-		(property "Notes" "Cost-down 2026-10-14 (was SRP5030T-3R3M): 3.3 uH, 38 mOhm max, Irms 5 A, Isat 8 A defined at a 40 % drop (not like-for-like with the SRP5030T); fine, as the 5.8 A IHS limit is a fault-only peak"
+		(property "Notes" "2026-10-30 (was APS0530M3R3H, 3.1 mm tall, hit the cup corner fillet at L502): ABC EHE05023R3MFB (JLC C49248023, in JLC stock), 5.5 x 5.2 x 2.0 mm max, 3.3 uH, 58 mOhm, Isat 5 A (30 %), 4.5 A rated; same electricals and land as COILMX MS0520-3R3M (C18163579, alternate). 2.0 mm height gives ~1.0 mm to the fillet. Isat is below the 5.8 A IHS limit, which is a fault-only peak. Footprint MonolithDev:L_COILMX_MS0520: land H 6.0, G 2.2, F 2.5 = 1.9 x 2.5 at +-2.05"
 			(at 128.27 203.2 0)
 			(hide yes)
@@
 			)
 		)
-		(property "LCSC" "C49073587"
+		(property "LCSC" "C49248023"
 			(at 128.27 203.2 0)
 			(hide yes)
@@
 			)
 		)
-		(property "MPN" "APS0530M3R3H (Coilank)"
+		(property "MPN" "EHE05023R3MFB (ABC)"
 			(at 128.27 203.2 0)
 			(hide yes)
